File: hardware/wah.sch (KiCad schematic (older format))
At the start: 21 parts, among them CON9 Jack_Stacked, U10 LM741

Commit message: Remove rescue lib dependency; Join gnd and gnda
Parts:
- D2: Manufacturer (none) -> Kingbright; Manufacturer Part Number (none) -> WP7113SRD/D; Supplier (none) -> Mouser; Supplier Link (none) -> http://www.mouser.de/ProductDetail/Kingbright/WP7113SRD-D/?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; Supplier Part Number (none) -> 604-WP7113SRD/D
Changed lines of the file:
@@
 F 1 "LED" H 6550 4950 50  0000 C CNN
 F 2 "" H 6550 5050 60  0000 C CNN
-F 3 "" H 6550 5050 60  0000 C CNN
+F 3 "http://www.kingbrightusa.com/images/catalog/SPEC/WP7113SRD-D.pdf" H 6550 5150 60  0001 C CNN
+F 4 "Mouser" H 6550 5150 60  0001 C CNN "Supplier"
+F 5 "604-WP7113SRD/D" H 6550 5150 60  0001 C CNN "Supplier Part Number"
+F 6 "http://www.mouser.de/ProductDetail/Kingbright/WP7113SRD-D/?qs=sGAEpiMZZMvHYEB9WUp7ElN5I0Rojjgy18duyl9iYGM%3d" H 6550 5150 60  0001 C CNN "Supplier Link"
+F 7 "Kingbright" H 6550 5150 60  0001 C CNN "Manufacturer"
+F 8 "WP7113SRD/D" H 6550 5150 60  0001 C CNN "Manufacturer Part Number"
 	1    6550 5050
 	0    1    1    0
