File: hardware/uMIDI-wah.sch (KiCad schematic (older format))
At the start: 29 parts

Commit message: Assign remaining footprints
Parts:
- C1, C4, C5, C8: renamed from C?; footprint (none) -> Capacitors_SMD:C_0603
- C10, C11, C12, C2, C6, C7, C9: renamed from C?; footprint (none) -> Capacitors_SMD:C_0805
- R2, R6: renamed from R?; footprint Resistors_SMD:R_0805 -> Resistors_SMD:R_0603
- R8: renamed from R?; footprint (none) -> Resistors_ThroughHole:Resistor_Horizontal_RM10mm
- gave numbers to parts that had none: 15

Commit message: Fix RV1 bom fields
Parts:
- RV1: Manufacturer Part Number http://www.bitechnologies.com/pdfs/23.pdf -> 23BR10KLFTR; Supplier Link http://www.mouser.de/Search/ProductDetail.aspx?qs=gQBTb7UQo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 -> http://www.mouser.de/ProductDetail/TT-Electronics/23BR10KLF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; Supplier Part Number 858-23BR10KLFTR -> 858-23BR10KLFTR
Changed lines of the file:
@@
 F 3 "http://www.bitechnologies.com/pdfs/23.pdf" H 7650 2900 60  0001 C CNN
 F 4 "Mouser" H 7650 2900 60  0001 C CNN "Supplier"
-F 5 "858-23BR10KLFTR " H 7650 2900 60  0001 C CNN "Supplier Part Number"
-F 6 "http://www.mouser.de/Search/ProductDetail.aspx?qs=gQBTb7UQo2KQtf18q%252b3T0Q%3d%3d" H 7650 2900 60  0001 C CNN "Supplier Link"
+F 5 "858-23BR10KLFTR" H 7650 2900 60  0001 C CNN "Supplier Part Number"
+F 6 "http://www.mouser.de/ProductDetail/TT-Electronics/23BR10KLFTR/?qs=%2fha2pyFaduiZ3ynuiECRXesjuD6u2n4EgsENysIu9nE8y5NJs6CTRA%3d%3d" H 7650 2900 60  0001 C CNN "Supplier Link"
 F 7 "TT electronics" H 7650 2900 60  0001 C CNN "Manufacturer"
-F 8 "http://www.bitechnologies.com/pdfs/23.pdf" H 7650 2900 60  0001 C CNN "Manufacturer Part Number"
+F 8 "23BR10KLFTR" H 7650 2900 60  0001 C CNN "Manufacturer Part Number"
 	1    7650 2900
 	0    1    1    0

Commit message: Add capacitor bom fields
Parts:
- C1, C4, C5, C8: footprint Capacitors_SMD:C_0603 -> Capacitors_SMD:C_0805; Manufacturer (none) -> Murata; Manufacturer Part Number (none) -> GRM21BR61E106KA73L; Supplier (none) -> Mouser; Supplier Link (none) -> http://eu.mouser.com/ProductDetail/Murata-Electronics/GRM21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; Supplier Part Number (none) -> 81-GRM21BR61E106KA3L
- C10: Manufacturer (none) -> Kemet; Manufacturer Part Number (none) -> C0805C509C5GACTU; Supplier (none) -> Mouser; Supplier Link (none) -> http://www.mouser.de/ProductDetail/Kemet/C0805C509C5GACTU/?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; Supplier Part Number (none) -> 80-C0805C509C5G
- C11: Manufacturer (none) -> Kemet; Manufacturer Part Number (none) -> C0805C202J3GACTU; Supplier (none) -> Mouser; Supplier Link (none) -> http://www.mouser.de/ProductDetail/Kemet/C0805C202J3GACTU/?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; Supplier Part Number (none) -> 80-C0805C202J3G
- C12, C2: Manufacturer (none) -> Kemet; Manufacturer Part Number (none) -> C0805C105K3RACTU; Supplier (none) -> Mouser; Supplier Link (none) -> http://www.mouser.de/ProductDetail/Kemet/C0805C105K3RACTU/?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; Supplier Part Number (none) -> 80-C0805C105K3R
- C6: Manufacturer (none) -> Murata; Manufacturer Part Number (none) -> GRM216R71H102KA01D; Supplier (none) -> Mouser; Supplier Link (none) -> http://www.mouser.de/ProductDetail/Murata-Electronics/GRM21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; Supplier Part Number (none) -> 81-GRM40X102K50D
- C7: Manufacturer (none) -> Murata; Manufacturer Part Number (none) -> GRM21BR71H473KA01L; Supplier (none) -> Mouser; Supplier Link (none) -> http://www.mouser.de/ProductDetail/Murata-Electronics/GRM21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; Supplier Part Number (none) -> 81-GRM40X473K50L
- C9: Manufacturer (none) -> Murata; Manufacturer Part Number (none) -> GRM21BR71H683KA01L; Supplier (none) -> Mouser; Supplier Link (none) -> http://www.mouser.de/ProductDetail/Murata-Electronics/GRM21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; Supplier Part Number (none) -> 81-GRM40X683K50L
Changed lines of the file:
@@
 F 1 "1n" V 5100 2300 50  0000 L CNN
 F 2 "Capacitors_SMD:C_0805" H 4988 2200 30  0001 C CNN
-F 3 "" H 4950 2350 60  0000 C CNN
+F 3 "http://psearch.en.murata.com/capacitor/product/GRM216R71H102KA01%23.pdf" H 4800 2300 60  0001 C CNN
+F 4 "Mouser" H 4800 2300 60  0001 C CNN "Supplier"
+F 5 "81-GRM40X102K50D" H 4800 2300 60  0001 C CNN "Supplier Part Number"
+F 6 "http://www.mouser.de/ProductDetail/Murata-Electronics/GRM216R71H102KA01D/?qs=sGAEpiMZZMs0AnBnWHyRQPmAk23g1ayjUUppCxLhx3E%3d" H 4800 2300 60  0001 C CNN "Supplier Link"
+F 7 "Murata" H 4800 2300 60  0001 C CNN "Manufacturer"
+F 8 "GRM216R71H102KA01D" H 4800 2300 60  0001 C CNN "Manufacturer Part Number"
 	1    4950 2350
 	0    1    1    0
@@
 F 1 "47n" V 5500 2550 50  0000 L CNN
 F 2 "Capacitors_SMD:C_0805" H 5388 2450 30  0001 C CNN
-F 3 "" H 5350 2600 60  0000 C CNN
+F 3 "http://psearch.en.murata.com/capacitor/product/GRM21BR71H473KA01%23.pdf" H 5200 2550 60  0001 C CNN
+F 4 "Mouser" H 5200 2550 60  0001 C CNN "Supplier"
+F 5 "81-GRM40X473K50L" H 5200 2550 60  0001 C CNN "Supplier Part Number"
+F 6 "http://www.mouser.de/ProductDetail/Murata-Electronics/GRM21BR71H473KA01L/?qs=sGAEpiMZZMs0AnBnWHyRQKf3b7LydMIhqNu%252bJe6zVN8%3d" H 5200 2550 60  0001 C CNN "Supplier Link"
+F 7 "Murata" H 5200 2550 60  0001 C CNN "Manufacturer"
+F 8 "GRM21BR71H473KA01L" H 5200 2550 60  0001 C CNN "Manufacturer Part Number"
 	1    5350 2600
 	0    1    1    0
@@
 F 0 "C8" H 5300 1400 50  0000 L CNN
 F 1 "10u" H 5250 1600 50  0000 L CNN
-F 2 "Capacitors_SMD:C_0603" H 5438 1350 30  0001 C CNN
-F 3 "" H 5400 1500 60  0000 C CNN
+F 2 "Capacitors_SMD:C_0805" H 5438 1350 30  0001 C CNN
+F 3 "http://psearch.en.murata.com/capacitor/product/GRM21BR61E106KA73%23.pdf" H 5300 1400 60  0001 C CNN
+F 4 "Mouser" H 5300 1400 60  0001 C CNN "Supplier"
+F 5 "81-GRM21BR61E106KA3L" H 5300 1400 60  0001 C CNN "Supplier Part Number"
+F 6 "http://eu.mouser.com/ProductDetail/Murata-Electronics/GRM21BR61E106KA73L/?qs=sGAEpiMZZMs0AnBnWHyRQEM2qvC6XUvU2imHfdddTY8%3d" H 5300 1400 60  0001 C CNN "Supplier Link"
+F 7 "Murata" H 5300 1400 60  0001 C CNN "Manufacturer"
+F 8 "GRM21BR61E106KA73L" H 5300 1400 60  0001 C CNN "Manufacturer Part Number"
 	1    5400 1500
 	-1   0    0    1
@@
 F 0 "C4" H 4250 1400 50  0000 L CNN
 F 1 "10u" H 4200 1600 50  0000 L CNN
-F 2 "Capacitors_SMD:C_0603" H 4388 1350 30  0001 C CNN
-F 3 "" H 4350 1500 60  0000 C CNN
+F 2 "Capacitors_SMD:C_0805" H 4388 1350 30  0001 C CNN
+F 3 "http://psearch.en.murata.com/capacitor/product/GRM21BR61E106KA73%23.pdf" H 4250 1400 60  0001 C CNN
+F 4 "Mouser" H 4250 1400 60  0001 C CNN "Supplier"
+F 5 "81-GRM21BR61E106KA3L" H 4250 1400 60  0001 C CNN "Supplier Part Number"
+F 6 "http://eu.mouser.com/ProductDetail/Murata-Electronics/GRM21BR61E106KA73L/?qs=sGAEpiMZZMs0AnBnWHyRQEM2qvC6XUvU2imHfdddTY8%3d" H 4250 1400 60  0001 C CNN "Supplier Link"
+F 7 "Murata" H 4250 1400 60  0001 C CNN "Manufacturer"
+F 8 "GRM21BR61E106KA73L" H 4250 1400 60  0001 C CNN "Manufacturer Part Number"
 	1    4350 1500
 	-1   0    0    1
@@
 F 0 "C5" H 4550 1400 50  0000 L CNN
 F 1 "10u" H 4500 1600 50  0000 L CNN
-F 2 "Capacitors_SMD:C_0603" H 4688 1350 30  0001 C CNN
-F 3 "" H 4650 1500 60  0000 C CNN
+F 2 "Capacitors_SMD:C_0805" H 4688 1350 30  0001 C CNN
+F 3 "http://psearch.en.murata.com/capacitor/product/GRM21BR61E106KA73%23.pdf" H 4550 1400 60  0001 C CNN
+F 4 "Mouser" H 4550 1400 60  0001 C CNN "Supplier"
+F 5 "81-GRM21BR61E106KA3L" H 4550 1400 60  0001 C CNN "Supplier Part Number"
+F 6 "http://eu.mouser.com/ProductDetail/Murata-Electronics/GRM21BR61E106KA73L/?qs=sGAEpiMZZMs0AnBnWHyRQEM2qvC6XUvU2imHfdddTY8%3d" H 4550 1400 60  0001 C CNN "Supplier Link"
+F 7 "Murata" H 4550 1400 60  0001 C CNN "Manufacturer"
+F 8 "GRM21BR61E106KA73L" H 4550 1400 60  0001 C CNN "Manufacturer Part Number"
 	1    4650 1500
 	-1   0    0    1
@@
 F 1 "5p" V 6300 3150 50  0000 L CNN
 F 2 "Capacitors_SMD:C_0805" H 6188 3050 30  0001 C CNN
-F 3 "" H 6150 3200 60  0000 C CNN
+F 3 "http://www.kemet.com/Lists/ProductCatalog/Attachments/46/KEM_C1003_C0G_SMD.pdf" H 6000 3150 60  0001 C CNN
+F 4 "Mouser" H 6000 3150 60  0001 C CNN "Supplier"
+F 5 "80-C0805C509C5G" H 6000 3150 60  0001 C CNN "Supplier Part Number"
+F 6 "http://www.mouser.de/ProductDetail/Kemet/C0805C509C5GACTU/?qs=sGAEpiMZZMs0AnBnWHyRQKp5FInkmPX89lHLVa%2ffUlM%3d" H 6000 3150 60  0001 C CNN "Supplier Link"
+F 7 "Kemet" H 6000 3150 60  0001 C CNN "Manufacturer"
+F 8 "C0805C509C5GACTU" H 6000 3150 60  0001 C CNN "Manufacturer Part Number"
 	1    6150 3200
 	0    1    1    0
@@
 F 1 "6.8n" H 5450 3750 50  0000 L CNN
 F 2 "Capacitors_SMD:C_0805" H 5688 3500 30  0001 C CNN
-F 3 "" H 5650 3650 60  0000 C CNN
+F 3 "http://psearch.en.murata.com/capacitor/product/GRM21BR71H683KA01%23.pdf" H 5550 3550 60  0001 C CNN
+F 4 "Mouser" H 5550 3550 60  0001 C CNN "Supplier"
+F 5 "81-GRM40X683K50L" H 5550 3550 60  0001 C CNN "Supplier Part Number"
+F 6 "http://www.mouser.de/ProductDetail/Murata-Electronics/GRM21BR71H683KA01L/?qs=sGAEpiMZZMs0AnBnWHyRQKf3b7LydMIhV8ZIV4K3K9k%3d" H 5550 3550 60  0001 C CNN "Supplier Link"
+F 7 "Murata" H 5550 3550 60  0001 C CNN "Manufacturer"
+F 8 "GRM21BR71H683KA01L" H 5550 3550 60  0001 C CNN "Manufacturer Part Number"
 	1    5650 3650
 	-1   0    0    1
@@
 F 1 "2n" H 6850 3750 50  0000 L CNN
 F 2 "Capacitors_SMD:C_0805" H 6988 3500 30  0001 C CNN
-F 3 "" H 6950 3650 60  0000 C CNN
+F 3 "http://www.kemet.com/Lists/ProductCatalog/Attachments/46/KEM_C1003_C0G_SMD.pdf" H 6850 3550 60  0001 C CNN
+F 4 "Mouser" H 6850 3550 60  0001 C CNN "Supplier"
+F 5 "80-C0805C202J3G" H 6850 3550 60  0001 C CNN "Supplier Part Number"
+F 6 "http://www.mouser.de/ProductDetail/Kemet/C0805C202J3GACTU/?qs=sGAEpiMZZMs0AnBnWHyRQCXsKWBJIgVSmQzlfJ9Rsqs%3d" H 6850 3550 60  0001 C CNN "Supplier Link"
+F 7 "Kemet" H 6850 3550 60  0001 C CNN "Manufacturer"
+F 8 "C0805C202J3GACTU" H 6850 3550 60  0001 C CNN "Manufacturer Part Number"
 	1    6950 3650
 	-1   0    0    1
@@
 F 1 "1u" V 7450 2450 50  0000 L CNN
 F 2 "Capacitors_SMD:C_0805" H 7338 2350 30  0001 C CNN
-F 3 "" H 7300 2500 60  0000 C CNN
+F 3 "http://www.kemet.com/Lists/ProductCatalog/Attachments/53/KEM_C1002_X7R_SMD.pdf" H 7150 2450 60  0001 C CNN
+F 4 "Mouser" H 7150 2450 60  0001 C CNN "Supplier"
+F 5 "80-C0805C105K3R" H 7150 2450 60  0001 C CNN "Supplier Part Number"
+F 6 "http://www.mouser.de/ProductDetail/Kemet/C0805C105K3RACTU/?qs=sGAEpiMZZMs0AnBnWHyRQHsuToI6krcdEBQqaF%2fNrvM%3d" H 7150 2450 60  0001 C CNN "Supplier Link"
+F 7 "Kemet" H 7150 2450 60  0001 C CNN "Manufacturer"
+F 8 "C0805C105K3RACTU" H 7150 2450 60  0001 C CNN "Manufacturer Part Number"
 	1    7300 2500
 	0    1    1    0
@@
 F 0 "C1" H 1400 1800 50  0000 L CNN
 F 1 "10u" H 1350 2000 50  0000 L CNN
-F 2 "Capacitors_SMD:C_0603" H 1538 1750 30  0001 C CNN
-F 3 "" H 1500 1900 60  0000 C CNN
+F 2 "Capacitors_SMD:C_0805" H 1538 1750 30  0001 C CNN
+F 3 "http://psearch.en.murata.com/capacitor/product/GRM21BR61E106KA73%23.pdf" H 1400 1800 60  0001 C CNN
+F 4 "Mouser" H 1400 1800 60  0001 C CNN "Supplier"
+F 5 "81-GRM21BR61E106KA3L" H 1400 1800 60  0001 C CNN "Supplier Part Number"
+F 6 "http://eu.mouser.com/ProductDetail/Murata-Electronics/GRM21BR61E106KA73L/?qs=sGAEpiMZZMs0AnBnWHyRQEM2qvC6XUvU2imHfdddTY8%3d" H 1400 1800 60  0001 C CNN "Supplier Link"
+F 7 "Murata" H 1400 1800 60  0001 C CNN "Manufacturer"
+F 8 "GRM21BR61E106KA73L" H 1400 1800 60  0001 C CNN "Manufacturer Part Number"
 	1    1500 1900
 	-1   0    0    1
@@
 F 1 "1u" H 1700 1800 50  0000 L CNN
 F 2 "Capacitors_SMD:C_0805" H 1738 1750 30  0001 C CNN
-F 3 "" H 1700 1900 60  0000 C CNN
+F 3 "http://www.kemet.com/Lists/ProductCatalog/Attachments/53/KEM_C1002_X7R_SMD.pdf" H 1700 2000 60  0001 C CNN
+F 4 "Mouser" H 1700 2000 60  0001 C CNN "Supplier"
+F 5 "80-C0805C105K3R" H 1700 2000 60  0001 C CNN "Supplier Part Number"
+F 6 "http://www.mouser.de/ProductDetail/Kemet/C0805C105K3RACTU/?qs=sGAEpiMZZMs0AnBnWHyRQHsuToI6krcdEBQqaF%2fNrvM%3d" H 1700 2000 60  0001 C CNN "Supplier Link"
+F 7 "Kemet" H 1700 2000 60  0001 C CNN "Manufacturer"
+F 8 "C0805C105K3RACTU" H 1700 2000 60  0001 C CNN "Manufacturer Part Number"
 	1    1700 1900
 	1    0    0    -1

Commit message: Add ldr bom fields; Change footprint
Parts:
- R8: value Photores -> LDR 05; footprint Resistors_ThroughHole:Resistor_Horizontal_RM10mm -> Capacitors_Elko_ThroughHole:Elko_vert_20x10mm_RM7.5; Supplier (none) -> Reichelt; Supplier Link (none) -> http://www.reichelt.de/LDR-05/3/index.html?&ACTION=3&LA=446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; Supplier Part Number (none) -> LDR 05
Changed lines of the file:
@@
 P 6350 4300
 F 0 "R8" V 6430 4300 50  0000 C CNN
-F 1 "Photores" V 6560 4300 50  0000 C TNN
-F 2 "Resistors_ThroughHole:Resistor_Horizontal_RM10mm" H 6280 4300 30  0001 C CNN
-F 3 "" H 6350 4300 30  0000 C CNN
+F 1 "LDR 05" V 6560 4300 50  0000 C TNN
+F 2 "Capacitors_Elko_ThroughHole:Elko_vert_20x10mm_RM7.5" H 6280 4300 30  0001 C CNN
+F 3 "http://cdn-reichelt.de/documents/datenblatt/A500/LDR05%23IMP.pdf" H 6430 4300 60  0001 C CNN
+F 4 "Reichelt" H 6430 4300 60  0001 C CNN "Supplier"
+F 5 "LDR 05" H 6430 4300 60  0001 C CNN "Supplier Part Number"
+F 6 "http://www.reichelt.de/LDR-05/3/index.html?&ACTION=3&LA=446&ARTICLE=10207&artnr=LDR+05&SEARCH=ldr05" H 6430 4300 60  0001 C CNN "Supplier Link"
 	1    6350 4300
 	1    0    0    -1

Commit message: Add resistor bom fields
Parts:
- R1, R3, R5: Manufacturer (none) -> Vishay/Dale; Manufacturer Part Number (none) -> CRCW0805100KFKEA; Supplier (none) -> Mouser; Supplier Link (none) -> http://www.mouser.de/ProductDetail/Vishay-Dale/CRCW0805100K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; Supplier Part Number (none) -> 71-CRCW0805-100K-E3
- R2, R6: Manufacturer (none) -> Vishay/Dale; Manufacturer Part Number (none) -> CRCW060382R0FKEA; Supplier (none) -> Mouser; Supplier Link (none) -> http://www.mouser.de/ProductDetail/Vishay-Dale/CRCW060382R0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; Supplier Part Number (none) -> 71-CRCW0603-82-E3
- R4: Manufacturer (none) -> Vishay/Dale; Manufacturer Part Number (none) -> CRCW080582K0FKEA; Supplier (none) -> Mouser; Supplier Link (none) -> http://www.mouser.de/Search/ProductDetail.aspx?qs=3kMMNJ4TL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; Supplier Part Number (none) -> 71-CRCW0805-82K-E3
- R7: Manufacturer (none) -> Vishay/Dale; Manufacturer Part Number (none) -> CRCW080510K0JNEA; Supplier (none) -> Mouser; Supplier Link (none) -> http://www.mouser.de/ProductDetail/Vishay-Dale/CRCW080510K0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; Supplier Part Number (none) -> 71-CRCW0805J-10K-E3
- R9: Manufacturer (none) -> Vishay/Dale; Manufacturer Part Number (none) -> CRCW08051M20FKEA; Supplier (none) -> Mouser; Supplier Link (none) -> http://www.mouser.de/ProductDetail/Vishay-Dale/CRCW08051M20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; Supplier Part Number (none) -> 71-CRCW08051M20FKEA
Changed lines of the file:
@@
 F 1 "100k" V 4557 2601 50  0000 C CNN
 F 2 "Resistors_SMD:R_0805" V 4480 2600 30  0001 C CNN
-F 3 "" H 4550 2600 30  0000 C CNN
+F 3 "http://www.vishay.com/docs/20022/dcrcwhe3.pdf" H 4450 2600 60  0001 C CNN
+F 4 "Mouser" H 4450 2600 60  0001 C CNN "Supplier"
+F 5 "71-CRCW0805-100K-E3" H 4450 2600 60  0001 C CNN "Supplier Part Number"
+F 6 "http://www.mouser.de/ProductDetail/Vishay-Dale/CRCW0805100KFKEA/?qs=sGAEpiMZZMtlubZbdhIBIKpw3Cj3Rl3MgRjH3xt31Ys%3d" H 4450 2600 60  0001 C CNN "Supplier Link"
+F 7 "Vishay/Dale" H 4450 2600 60  0001 C CNN "Manufacturer"
+F 8 "CRCW0805100KFKEA" H 4450 2600 60  0001 C CNN "Manufacturer Part Number"
 	1    4550 2600
 	0    1    1    0
@@
 F 1 "82k" V 4957 2601 50  0000 C CNN
 F 2 "Resistors_SMD:R_0805" V 4880 2600 30  0001 C CNN
-F 3 "" H 4950 2600 30  0000 C CNN
+F 3 "http://www.vishay.com/docs/20022/dcrcwhe3.pdf" H 5050 2600 60  0001 C CNN
+F 4 "Mouser" H 5050 2600 60  0001 C CNN "Supplier"
+F 5 "71-CRCW0805-82K-E3" H 5050 2600 60  0001 C CNN "Supplier Part Number"
+F 6 "http://www.mouser.de/Search/ProductDetail.aspx?qs=3kMMNJ4TLu3mlayDxFJc8A%3d%3d" H 5050 2600 60  0001 C CNN "Supplier Link"
+F 7 "Vishay/Dale" H 5050 2600 60  0001 C CNN "Manufacturer"
+F 8 "CRCW080582K0FKEA" H 5050 2600 60  0001 C CNN "Manufacturer Part Number"
 	1    4950 2600
 	0    1    1    0
@@
 F 1 "100k" V 4857 1301 50  0000 C CNN
 F 2 "Resistors_SMD:R_0805" V 4780 1300 30  0001 C CNN
-F 3 "" H 4850 1300 30  0000 C CNN
+F 3 "http://www.vishay.com/docs/20022/dcrcwhe3.pdf" H 4930 1300 60  0001 C CNN
+F 4 "Mouser" H 4930 1300 60  0001 C CNN "Supplier"
+F 5 "71-CRCW0805-100K-E3" H 4930 1300 60  0001 C CNN "Supplier Part Number"
+F 6 "http://www.mouser.de/ProductDetail/Vishay-Dale/CRCW0805100KFKEA/?qs=sGAEpiMZZMtlubZbdhIBIKpw3Cj3Rl3MgRjH3xt31Ys%3d" H 4930 1300 60  0001 C CNN "Supplier Link"
+F 7 "Vishay/Dale" H 4930 1300 60  0001 C CNN "Manufacturer"
+F 8 "CRCW0805100KFKEA" H 4930 1300 60  0001 C CNN "Manufacturer Part Number"
 	1    4850 1300
 	0    -1   -1   0
@@
 F 1 "100k" V 5107 1501 50  0000 C CNN
 F 2 "Resistors_SMD:R_0805" V 5030 1500 30  0001 C CNN
-F 3 "" H 5100 1500 30  0000 C CNN
+F 3 "http://www.vishay.com/docs/20022/dcrcwhe3.pdf" H 5180 1500 60  0001 C CNN
+F 4 "Mouser" H 5180 1500 60  0001 C CNN "Supplier"
+F 5 "71-CRCW0805-100K-E3" H 5180 1500 60  0001 C CNN "Supplier Part Number"
+F 6 "http://www.mouser.de/ProductDetail/Vishay-Dale/CRCW0805100KFKEA/?qs=sGAEpiMZZMtlubZbdhIBIKpw3Cj3Rl3MgRjH3xt31Ys%3d" H 5180 1500 60  0001 C CNN "Supplier Link"
+F 7 "Vishay/Dale" H 5180 1500 60  0001 C CNN "Manufacturer"
+F 8 "CRCW0805100KFKEA" H 5180 1500 60  0001 C CNN "Manufacturer Part Number"
 	1    5100 1500
 	1    0    0    -1
@@
 F 1 "1.2M" V 6507 3201 50  0000 C CNN
 F 2 "Resistors_SMD:R_0805" V 6430 3200 30  0001 C CNN
-F 3 "" H 6500 3200 30  0000 C CNN
+F 3 "http://www.vishay.com/docs/20022/dcrcwhe3.pdf" H 6400 3200 60  0001 C CNN
+F 4 "Mouser" H 6400 3200 60  0001 C CNN "Supplier"
+F 5 "71-CRCW08051M20FKEA" H 6400 3200 60  0001 C CNN "Supplier Part Number"
+F 6 "http://www.mouser.de/ProductDetail/Vishay-Dale/CRCW08051M20FKEA/?qs=sGAEpiMZZMu61qfTUdNhG%2fIq7AJBeSZM%2fAynCVp7nNM%3d" H 6400 3200 60  0001 C CNN "Supplier Link"
+F 7 "Vishay/Dale" H 6400 3200 60  0001 C CNN "Manufacturer"
+F 8 "CRCW08051M20FKEA" H 6400 3200 60  0001 C CNN "Manufacturer Part Number"
 	1    6500 3200
 	0    1    1    0
@@
 F 1 "470k" V 6357 3451 50  0000 C CNN
 F 2 "Resistors_SMD:R_0805" V 6280 3450 30  0001 C CNN
-F 3 "" H 6350 3450 30  0000 C CNN
+F 3 "http://www.vishay.com/docs/20022/dcrcwhe3.pdf" H 6250 3450 60  0001 C CNN
+F 4 "Mouser" H 6250 3450 60  0001 C CNN "Supplier"
+F 5 "71-CRCW0805J-10K-E3" H 6250 3450 60  0001 C CNN "Supplier Part Number"
+F 6 "http://www.mouser.de/ProductDetail/Vishay-Dale/CRCW080510K0JNEA/?qs=sGAEpiMZZMu61qfTUdNhG2DpbjADlD3G7HGBoM9TRSM%3d" H 6250 3450 60  0001 C CNN "Supplier Link"
+F 7 "Vishay/Dale" H 6250 3450 60  0001 C CNN "Manufacturer"
+F 8 "CRCW080510K0JNEA" H 6250 3450 60  0001 C CNN "Manufacturer Part Number"
 	1    6350 3450
 	0    1    1    0
@@
 F 1 "82" V 5707 4051 50  0000 C CNN
 F 2 "Resistors_SMD:R_0603" V 5630 4050 30  0001 C CNN
-F 3 "" H 5700 4050 30  0000 C CNN
+F 3 "http://www.vishay.com/docs/20022/dcrcwhe3.pdf" H 5780 4050 60  0001 C CNN
+F 4 "Mouser" H 5780 4050 60  0001 C CNN "Supplier"
+F 5 "71-CRCW0603-82-E3" H 5780 4050 60  0001 C CNN "Supplier Part Number"
+F 6 "http://www.mouser.de/ProductDetail/Vishay-Dale/CRCW060382R0FKEA/?qs=sGAEpiMZZMu61qfTUdNhG3XwnH6YDjgjsOpBFaxMcQ0%3d" H 5780 4050 60  0001 C CNN "Supplier Link"
+F 7 "Vishay/Dale" H 5780 4050 60  0001 C CNN "Manufacturer"
+F 8 "CRCW060382R0FKEA" H 5780 4050 60  0001 C CNN "Manufacturer Part Number"
 	1    5700 4050
 	0    1    1    0
@@
 F 1 "82" V 4757 5601 50  0000 C CNN
 F 2 "Resistors_SMD:R_0603" V 4680 5600 30  0001 C CNN
-F 3 "" H 4750 5600 30  0000 C CNN
+F 3 "http://www.vishay.com/docs/20022/dcrcwhe3.pdf" H 4830 5600 60  0001 C CNN
+F 4 "Mouser" H 4830 5600 60  0001 C CNN "Supplier"
+F 5 "71-CRCW0603-82-E3" H 4830 5600 60  0001 C CNN "Supplier Part Number"
+F 6 "http://www.mouser.de/ProductDetail/Vishay-Dale/CRCW060382R0FKEA/?qs=sGAEpiMZZMu61qfTUdNhG3XwnH6YDjgjsOpBFaxMcQ0%3d" H 4830 5600 60  0001 C CNN "Supplier Link"
+F 7 "Vishay/Dale" H 4830 5600 60  0001 C CNN "Manufacturer"
+F 8 "CRCW060382R0FKEA" H 4830 5600 60  0001 C CNN "Manufacturer Part Number"
 	1    4750 5600
 	-1   0    0    1
