File: hardware/uMIDI-wah.sch (KiCad schematic (older format))
At the start: 24 parts, among them U1 Opamp_Dual_Generic, X1 AudioJack3_Switch

Commit message: Annotate schematic
Parts:
- L1: footprint (none) -> Inductor_THT:L_Toroid_Horizontal_D17.3mm_P15.24mm_Bourns_2000
- R4: footprint (none) -> Resistor_SMD:R_0805_2012Metric_Pad1.15x1.40mm_HandSolder
- gave numbers to parts that had none: 12
Changed lines of the file:
@@
 F 0 "R4" H 3770 4146 50  0000 L CNN
 F 1 "1k" H 3770 4055 50  0000 L CNN
-F 2 "" V 3630 4100 50  0001 C CNN
+F 2 "Resistor_SMD:R_0805_2012Metric_Pad1.15x1.40mm_HandSolder" V 3630 4100 50  0001 C CNN
 F 3 "~" H 3700 4100 50  0001 C CNN
 	1    3700 4100
@@
 F 0 "L1" H 3753 4946 50  0000 L CNN
 F 1 "500m" H 3753 4855 50  0000 L CNN
-F 2 "" H 3700 4900 50  0001 C CNN
+F 2 "Inductor_THT:L_Toroid_Horizontal_D17.3mm_P15.24mm_Bourns_2000" H 3700 4900 50  0001 C CNN
 F 3 "~" H 3700 4900 50  0001 C CNN
 	1    3700 4900
@@
 	5700 4650 5700 5100
 $Comp
-L power:GND #PWR?
+L power:GND #PWR07
 U 1 1 5C88B808
 P 5700 5100
-F 0 "#PWR?" H 5700 4850 50  0001 C CNN
+F 0 "#PWR07" H 5700 4850 50  0001 C CNN
 F 1 "GND" H 5705 4927 50  0000 C CNN
 F 2 "" H 5700 5100 50  0001 C CNN
@@
 $EndComp
 $Comp
-L Sensor_Optical:LDR07 R?
+L Sensor_Optical:LDR07 R5
 U 1 1 5C8C34D2
 P 3350 4900
-F 0 "R?" H 3420 4946 50  0000 L CNN
+F 0 "R5" H 3420 4946 50  0000 L CNN
 F 1 "LDR07" H 3420 4855 50  0000 L CNN
 F 2 "OptoDevice:R_LDR_5.1x4.3mm_P3.4mm_Vertical" V 3525 4900 50  0001 C CNN
@@
 $EndComp
 $Comp
-L Sensor_Optical:LDR07 R?
+L Sensor_Optical:LDR07 R9
 U 1 1 5C8C3558
 P 6600 4850
-F 0 "R?" H 6412 4896 50  0000 R CNN
+F 0 "R9" H 6412 4896 50  0000 R CNN
 F 1 "LDR07" H 6412 4805 50  0000 R CNN
 F 2 "OptoDevice:R_LDR_5.1x4.3mm_P3.4mm_Vertical" V 6775 4850 50  0001 C CNN
@@
 	3350 4550 3700 4550
 $Comp
-L power:GND #PWR?
+L power:GND #PWR01
 U 1 1 5C8C493C
 P 2700 2600
-F 0 "#PWR?" H 2700 2350 50  0001 C CNN
+F 0 "#PWR01" H 2700 2350 50  0001 C CNN
 F 1 "GND" H 2705 2427 50  0000 C CNN
 F 2 "" H 2700 2600 50  0001 C CNN
@@
 Connection ~ 6600 4450
 $Comp
-L power:GND #PWR?
+L power:GND #PWR011
 U 1 1 5C8C63F2
 P 6600 5100
-F 0 "#PWR?" H 6600 4850 50  0001 C CNN
+F 0 "#PWR011" H 6600 4850 50  0001 C CNN
 F 1 "GND" H 6605 4927 50  0000 C CNN
 F 2 "" H 6600 5100 50  0001 C CNN
@@
 	6600 5100 6600 5000
 $Comp
-L power:GND #PWR?
+L power:GND #PWR03
 U 1 1 5C8C6D5F
 P 3350 5100
-F 0 "#PWR?" H 3350 4850 50  0001 C CNN
+F 0 "#PWR03" H 3350 4850 50  0001 C CNN
 F 1 "GND" H 3355 4927 50  0000 C CNN
 F 2 "" H 3350 5100 50  0001 C CNN
@@
 $EndComp
 $Comp
-L power:GND #PWR?
+L power:GND #PWR05
 U 1 1 5C8C6D8C
 P 3700 5100
-F 0 "#PWR?" H 3700 4850 50  0001 C CNN
+F 0 "#PWR05" H 3700 4850 50  0001 C CNN
 F 1 "GND" H 3705 4927 50  0000 C CNN
 F 2 "" H 3700 5100 50  0001 C CNN
@@
 	3700 5100 3700 5050
 $Comp
-L Device:C C?
+L Device:C C1
 U 1 1 5C8C9B22
 P 2750 3300
-F 0 "C?" V 2498 3300 50  0000 C CNN
+F 0 "C1" V 2498 3300 50  0000 C CNN
 F 1 "220u" V 2589 3300 50  0000 C CNN
 F 2 "" H 2788 3150 50  0001 C CNN
@@
 $EndComp
 $Comp
-L Connector:AudioJack3_Switch X?
+L Connector:AudioJack3_Switch X3
 U 1 1 5C8CAC4B
 P 6400 950
-F 0 "X?" H 6167 971 50  0000 R CNN
+F 0 "X3" H 6167 971 50  0000 R CNN
 F 1 "AudioJack3_Switch" H 6167 880 50  0000 R CNN
 F 2 "" H 6400 950 50  0001 C CNN
@@
 $EndComp
 $Comp
-L Device:R R?
+L Device:R R10
 U 1 1 5C8CF6D3
 P 3250 1450
-F 0 "R?" V 3043 1450 50  0000 C CNN
+F 0 "R10" V 3043 1450 50  0000 C CNN
 F 1 "1M" V 3134 1450 50  0000 C CNN
 F 2 "" V 3180 1450 50  0001 C CNN
@@
 	3500 1550 3500 1450
 $Comp
-L power:GND #PWR?
+L power:GND #PWR04
 U 1 1 5C8CC597
 P 3500 1550
-F 0 "#PWR?" H 3500 1300 50  0001 C CNN
+F 0 "#PWR04" H 3500 1300 50  0001 C CNN
 F 1 "GND" H 3505 1377 50  0000 C CNN
 F 2 "" H 3500 1550 50  0001 C CNN
@@
 	3400 1450 3500 1450
 $Comp
-L power:GND #PWR?
+L power:GND #PWR02
 U 1 1 5C8D511F
 P 3100 1050
-F 0 "#PWR?" H 3100 800 50  0001 C CNN
+F 0 "#PWR02" H 3100 800 50  0001 C CNN
 F 1 "GND" H 3105 877 50  0000 C CNN
 F 2 "" H 3100 1050 50  0001 C CNN
@@
 	6300 4450 6600 4450
 $Comp
-L Device:R_POT_TRIM RV?
+L Device:R_POT_TRIM RV1
 U 1 1 5CCE08C7
 P 5250 3650
-F 0 "RV?" V 5550 3850 50  0000 R CNN
+F 0 "RV1" V 5550 3850 50  0000 R CNN
 F 1 "470k" V 5500 3850 50  0000 R CNN
 F 2 "" H 5250 3650 50  0001 C CNN
@@
 Connection ~ 5700 3950
 $Comp
-L Device:R_POT_TRIM RV?
+L Device:R_POT_TRIM RV3
 U 1 1 5CCF56CF
 P 7550 3450
-F 0 "RV?" V 7850 3650 50  0000 R CNN
+F 0 "RV3" V 7850 3650 50  0000 R CNN
 F 1 "10k" V 7800 3650 50  0000 R CNN
 F 2 "" H 7550 3450 50  0001 C CNN
@@
 	7550 3600 7550 3650
 $Comp
-L power:GND #PWR?
+L power:GND #PWR012
 U 1 1 5CCF7EC5
 P 7550 3650
-F 0 "#PWR?" H 7550 3400 50  0001 C CNN
+F 0 "#PWR012" H 7550 3400 50  0001 C CNN
 F 1 "GND" H 7555 3477 50  0000 C CNN
 F 2 "" H 7550 3650 50  0001 C CNN
@@
 	6150 1250 6200 1250
 $Comp
-L Device:R R?
+L Device:R R11
 U 1 1 5CD0241C
 P 6350 1600
-F 0 "R?" V 6143 1600 50  0000 C CNN
+F 0 "R11" V 6143 1600 50  0000 C CNN
 F 1 "1M" V 6234 1600 50  0000 C CNN
 F 2 "" V 6280 1600 50  0001 C CNN
@@
 	6600 1700 6600 1600
 $Comp
-L power:GND #PWR?
+L power:GND #PWR010
 U 1 1 5CD02427
 P 6600 1700
-F 0 "#PWR?" H 6600 1450 50  0001 C CNN
+F 0 "#PWR010" H 6600 1450 50  0001 C CNN
 F 1 "GND" H 6605 1527 50  0000 C CNN
 F 2 "" H 6600 1700 50  0001 C CNN
@@
 	6150 1250 6150 1600
 $Comp
-L Device:R_POT_TRIM RV?
+L Device:R_POT_TRIM RV2
 U 1 1 5CD094F7
 P 6300 3750
-F 0 "RV?" V 6600 3950 50  0000 R CNN
+F 0 "RV2" V 6600 3950 50  0000 R CNN
 F 1 "470k" V 6550 3950 50  0000 R CNN
 F 2 "" H 6300 3750 50  0001 C CNN
@@
 	6600 4000 6600 3900
 $Comp
-L Connector_Generic:Conn_01x08 X?
+L Connector_Generic:Conn_01x08 X2
 U 1 1 5CD13F79
 P 4600 6300
-F 0 "X?" H 4680 6292 50  0000 L CNN
+F 0 "X2" H 4680 6292 50  0000 L CNN
 F 1 "Conn_01x08" H 4680 6201 50  0000 L CNN
 F 2 "" H 4600 6300 50  0001 C CNN
@@
 $EndComp
 $Comp
-L Device:C C?
+L Device:C C3
 U 1 1 5CD145B7
 P 6100 6350
-F 0 "C?" V 5848 6350 50  0000 C CNN
+F 0 "C3" V 5848 6350 50  0000 C CNN
 F 1 "100n" V 5939 6350 50  0000 C CNN
 F 2 "" H 6138 6200 50  0001 C CNN
@@
 $EndComp
 $Comp
-L Device:C C?
+L Device:C C2
 U 1 1 5CD147F0
 P 5700 6350
-F 0 "C?" V 5448 6350 50  0000 C CNN
+F 0 "C2" V 5448 6350 50  0000 C CNN
 F 1 "10u" V 5539 6350 50  0000 C CNN
 F 2 "" H 5738 6200 50  0001 C CNN
@@
 LED_Supply
 $Comp
-L power:GND #PWR?
+L power:GND #PWR06
 U 1 1 5CD38D2A
 P 4250 6950
-F 0 "#PWR?" H 4250 6700 50  0001 C CNN
+F 0 "#PWR06" H 4250 6700 50  0001 C CNN
 F 1 "GND" H 4255 6777 50  0000 C CNN
 F 2 "" H 4250 6950 50  0001 C CNN
@@
 VDDa
 $Comp
-L power:GND #PWR?
+L power:GND #PWR08
 U 1 1 5CD473BB
 P 5700 6850
-F 0 "#PWR?" H 5700 6600 50  0001 C CNN
+F 0 "#PWR08" H 5700 6600 50  0001 C CNN
 F 1 "GND" H 5705 6677 50  0000 C CNN
 F 2 "" H 5700 6850 50  0001 C CNN
@@
 	5650 1150 6200 1150
 $Comp
-L power:GND #PWR?
+L power:GND #PWR09
 U 1 1 5CDC7574
 P 6100 1050
-F 0 "#PWR?" H 6100 800 50  0001 C CNN
+F 0 "#PWR09" H 6100 800 50  0001 C CNN
 F 1 "GND" H 6105 877 50  0000 C CNN
 F 2 "" H 6100 1050 50  0001 C CNN

Commit message: Use 0805 footprint for all resistors
Parts:
- R1, R10, R11, R2, R3, R6, R7, R8: footprint (none) -> Resistors_SMD:R_0805
- R4: footprint Resistor_SMD:R_0805_2012Metric_Pad1.15x1.40mm_HandSolder -> Resistors_SMD:R_0805
- R5, R9: footprint OptoDevice:R_LDR_5.1x4.3mm_P3.4mm_Vertical -> Resistors_SMD:R_0805
Changed lines of the file:
@@
 F 0 "R2" V 3043 2600 50  0000 C CNN
 F 1 "1k" V 3134 2600 50  0000 C CNN
-F 2 "" V 3180 2600 50  0001 C CNN
-F 3 "~" H 3250 2600 50  0001 C CNN
+F 2 "Resistors_SMD:R_0805" V 3180 2600 50  0001 C CNN
+F 3 "" H 3250 2600 50  0001 C CNN
 	1    3250 2600
 	0    1    1    0
@@
 F 0 "R1" V 3457 3300 50  0000 C CNN
 F 1 "100k" V 3366 3300 50  0000 C CNN
-F 2 "" V 3180 3300 50  0001 C CNN
-F 3 "~" H 3250 3300 50  0001 C CNN
+F 2 "Resistors_SMD:R_0805" V 3180 3300 50  0001 C CNN
+F 3 "" H 3250 3300 50  0001 C CNN
 	1    3250 3300
 	0    1    -1   0
@@
 F 0 "R4" H 3770 4146 50  0000 L CNN
 F 1 "1k" H 3770 4055 50  0000 L CNN
-F 2 "Resistor_SMD:R_0805_2012Metric_Pad1.15x1.40mm_HandSolder" V 3630 4100 50  0001 C CNN
-F 3 "~" H 3700 4100 50  0001 C CNN
+F 2 "Resistors_SMD:R_0805" V 3630 4100 50  0001 C CNN
+F 3 "" H 3700 4100 50  0001 C CNN
 	1    3700 4100
 	1    0    0    -1
@@
 F 0 "R8" V 6357 4450 50  0000 C CNN
 F 1 "100k" V 6266 4450 50  0000 C CNN
-F 2 "" V 6080 4450 50  0001 C CNN
-F 3 "~" H 6150 4450 50  0001 C CNN
+F 2 "Resistors_SMD:R_0805" V 6080 4450 50  0001 C CNN
+F 3 "" H 6150 4450 50  0001 C CNN
 	1    6150 4450
 	0    1    -1   0
@@
 F 0 "R7" H 6670 3796 50  0000 L CNN
 F 1 "dnf" H 6670 3705 50  0000 L CNN
-F 2 "" V 6530 3750 50  0001 C CNN
-F 3 "~" H 6600 3750 50  0001 C CNN
+F 2 "Resistors_SMD:R_0805" V 6530 3750 50  0001 C CNN
+F 3 "" H 6600 3750 50  0001 C CNN
 	1    6600 3750
 	1    0    0    -1
@@
 F 0 "R3" V 3943 2600 50  0000 C CNN
 F 1 "100k" V 4034 2600 50  0000 C CNN
-F 2 "" V 4080 2600 50  0001 C CNN
-F 3 "~" H 4150 2600 50  0001 C CNN
+F 2 "Resistors_SMD:R_0805" V 4080 2600 50  0001 C CNN
+F 3 "" H 4150 2600 50  0001 C CNN
 	1    4150 2600
 	0    1    1    0
@@
 F 0 "R6" V 5350 3850 50  0000 C CNN
 F 1 "dnf" V 5350 4000 50  0000 C CNN
-F 2 "" V 5180 3950 50  0001 C CNN
-F 3 "~" H 5250 3950 50  0001 C CNN
+F 2 "Resistors_SMD:R_0805" V 5180 3950 50  0001 C CNN
+F 3 "" H 5250 3950 50  0001 C CNN
 	1    5250 3950
 	0    1    -1   0
@@
 F 0 "R5" H 3420 4946 50  0000 L CNN
 F 1 "LDR07" H 3420 4855 50  0000 L CNN
-F 2 "OptoDevice:R_LDR_5.1x4.3mm_P3.4mm_Vertical" V 3525 4900 50  0001 C CNN
-F 3 "http://www.tme.eu/de/Document/f2e3ad76a925811312d226c31da4cd7e/LDR07.pdf" H 3350 4850 50  0001 C CNN
+F 2 "Resistors_SMD:R_0805" V 3525 4900 50  0001 C CNN
+F 3 "" H 3350 4850 50  0001 C CNN
 	1    3350 4900
 	1    0    0    -1
@@
 F 0 "R9" H 6412 4896 50  0000 R CNN
 F 1 "LDR07" H 6412 4805 50  0000 R CNN
-F 2 "OptoDevice:R_LDR_5.1x4.3mm_P3.4mm_Vertical" V 6775 4850 50  0001 C CNN
-F 3 "http://www.tme.eu/de/Document/f2e3ad76a925811312d226c31da4cd7e/LDR07.pdf" H 6600 4800 50  0001 C CNN
+F 2 "Resistors_SMD:R_0805" V 6775 4850 50  0001 C CNN
+F 3 "" H 6600 4800 50  0001 C CNN
 	1    6600 4850
 	-1   0    0    -1
@@
 F 0 "R10" V 3043 1450 50  0000 C CNN
 F 1 "1M" V 3134 1450 50  0000 C CNN
-F 2 "" V 3180 1450 50  0001 C CNN
-F 3 "~" H 3250 1450 50  0001 C CNN
+F 2 "Resistors_SMD:R_0805" V 3180 1450 50  0001 C CNN
+F 3 "" H 3250 1450 50  0001 C CNN
 	1    3250 1450
 	0    1    1    0
@@
 F 0 "R11" V 6143 1600 50  0000 C CNN
 F 1 "1M" V 6234 1600 50  0000 C CNN
-F 2 "" V 6280 1600 50  0001 C CNN
-F 3 "~" H 6350 1600 50  0001 C CNN
+F 2 "Resistors_SMD:R_0805" V 6280 1600 50  0001 C CNN
+F 3 "" H 6350 1600 50  0001 C CNN
 	1    6350 1600
 	0    1    1    0

Commit message: Use 0805 footprint for all capacitors
Parts:
- C1, C2, C3, C4, C6: footprint (none) -> Capacitors_SMD:C_0805
Changed lines of the file:
@@
 F 0 "C6" V 6798 3200 50  0000 C CNN
 F 1 "220u" V 6889 3200 50  0000 C CNN
-F 2 "" H 7088 3050 50  0001 C CNN
-F 3 "~" H 7050 3200 50  0001 C CNN
+F 2 "Capacitors_SMD:C_0805" H 7088 3050 50  0001 C CNN
+F 3 "" H 7050 3200 50  0001 C CNN
 	1    7050 3200
 	0    1    1    0
@@
 F 0 "C4" V 3998 4550 50  0000 C CNN
 F 1 "33n" V 4089 4550 50  0000 C CNN
-F 2 "" H 4288 4400 50  0001 C CNN
-F 3 "~" H 4250 4550 50  0001 C CNN
+F 2 "Capacitors_SMD:C_0805" H 4288 4400 50  0001 C CNN
+F 3 "" H 4250 4550 50  0001 C CNN
 	1    4250 4550
 	0    1    1    0
@@
 F 0 "C1" V 2498 3300 50  0000 C CNN
 F 1 "220u" V 2589 3300 50  0000 C CNN
-F 2 "" H 2788 3150 50  0001 C CNN
-F 3 "~" H 2750 3300 50  0001 C CNN
+F 2 "Capacitors_SMD:C_0805" H 2788 3150 50  0001 C CNN
+F 3 "" H 2750 3300 50  0001 C CNN
 	1    2750 3300
 	0    1    1    0
@@
 F 0 "C3" V 5848 6350 50  0000 C CNN
 F 1 "100n" V 5939 6350 50  0000 C CNN
-F 2 "" H 6138 6200 50  0001 C CNN
-F 3 "~" H 6100 6350 50  0001 C CNN
+F 2 "Capacitors_SMD:C_0805" H 6138 6200 50  0001 C CNN
+F 3 "" H 6100 6350 50  0001 C CNN
 	1    6100 6350
 	-1   0    0    1
@@
 F 0 "C2" V 5448 6350 50  0000 C CNN
 F 1 "10u" V 5539 6350 50  0000 C CNN
-F 2 "" H 5738 6200 50  0001 C CNN
-F 3 "~" H 5700 6350 50  0001 C CNN
+F 2 "Capacitors_SMD:C_0805" H 5738 6200 50  0001 C CNN
+F 3 "" H 5700 6350 50  0001 C CNN
 	1    5700 6350
 	-1   0    0    1

Commit message: Add seconde fasel and Vref circuit
Parts:
- removed C2: 10u, Capacitors_SMD:C_0805, symbol Device:C
- added C12: 22u, Capacitors_SMD:C_0805, symbol Device:C
- added C2: 100u, 50V, Capacitor_SMD:CP_Elec_6.3x9.9, symbol Device:CP
- added D4: D, Diode_SMD:D_SMA-SMB_Universal_Handsoldering, symbol Device:D
- added L2: Fasel Yellow, Inductor_THT:L_Toroid_Horizontal_D17.3mm_P15.24mm_Bourns_2000, symbol Device:L
- added R21, R22: 100k, Resistors_SMD:R_0805, symbol Device:R
- added SW? (x2): SW_DPDT_x2, symbol Switch:SW_DPDT_x2
- C1, C6: value 220u -> 22u
- L1: value 500m -> Fasel Red
Connections:
- net GND: now also C12.1, C2.2, R22.1; no longer L1.2, R2.2, R5.2, R9.2, U1.5 (+)
- net VDDa: now also C2.1, D4.1 (K), R21.2; no longer X2.7 (Pin_7)
- net q: now also SW?.5 (B); no longer L1.1
- new net: L1.1, SW?.4 (A)
- new net: L1.2, SW?.1 (A)
- new net: D4.2 (A), X2.7 (Pin_7)
- new net: L2.2, SW?.3 (C)
- new net: L2.1, SW?.6 (C)
- new net Vref: C12.2, R2.2, R21.1, R22.2, R5.2, R9.2, SW?.2 (B), U1.5 (+)
Other:
- moved on the sheet: C3, L1, R5, U1C, X2

Commit message: Select and set all pots to 470k
Parts:
- RV1, RV2: Manufacturer (none) -> Vishay; Manufacturer Part Number (none) -> T7YA474MT20; Supplier (none) -> RS; Supplier Link (none) -> https://de.rs-online.com/web/p/abgleichwiderstande/3746844/; Supplier Part Number (none) -> 374-6844
- RV3: value 10k -> 470k; Manufacturer (none) -> Vishay; Manufacturer Part Number (none) -> T7YA474MT20; Supplier (none) -> RS; Supplier Link (none) -> https://de.rs-online.com/web/p/abgleichwiderstande/3746844/; Supplier Part Number (none) -> 374-6844
- SW? (x2): Manufacturer (none) -> TE; Manufacturer Part Number (none) -> 1825163-1; Supplier (none) -> RS; Supplier Link (none) -> https://de.rs-online.com/web/p/schiebeschalter/7455820/; Supplier Part Number (none) -> 745-5820
Changed lines of the file:
@@
 F 2 "" H 5250 3650 50  0001 C CNN
 F 3 "~" H 5250 3650 50  0001 C CNN
+F 4 "RS" V 5550 3850 50  0001 R CNN "Supplier"
+F 5 "374-6844" V 5550 3850 50  0001 R CNN "Supplier Part Number"
+F 6 "https://de.rs-online.com/web/p/abgleichwiderstande/3746844/" V 5550 3850 50  0001 R CNN "Supplier Link"
+F 7 "Vishay" V 5550 3850 50  0001 R CNN "Manufacturer"
+F 8 "T7YA474MT20" V 5550 3850 50  0001 R CNN "Manufacturer Part Number"
 	1    5250 3650
 	0    -1   -1   0
@@
 P 7550 3450
 F 0 "RV3" V 7850 3650 50  0000 R CNN
-F 1 "10k" V 7800 3650 50  0000 R CNN
+F 1 "470k" V 7800 3650 50  0000 R CNN
 F 2 "" H 7550 3450 50  0001 C CNN
 F 3 "~" H 7550 3450 50  0001 C CNN
+F 4 "RS" V 7850 3650 50  0001 R CNN "Supplier"
+F 5 "374-6844" V 7850 3650 50  0001 R CNN "Supplier Part Number"
+F 6 "https://de.rs-online.com/web/p/abgleichwiderstande/3746844/" V 7850 3650 50  0001 R CNN "Supplier Link"
+F 7 "Vishay" V 7850 3650 50  0001 R CNN "Manufacturer"
+F 8 "T7YA474MT20" V 7850 3650 50  0001 R CNN "Manufacturer Part Number"
 	1    7550 3450
 	1    0    0    -1
@@
 F 2 "" H 6300 3750 50  0001 C CNN
 F 3 "~" H 6300 3750 50  0001 C CNN
+F 4 "RS" V 6600 3950 50  0001 R CNN "Supplier"
+F 5 "374-6844" V 6600 3950 50  0001 R CNN "Supplier Part Number"
+F 6 "https://de.rs-online.com/web/p/abgleichwiderstande/3746844/" V 6600 3950 50  0001 R CNN "Supplier Link"
+F 7 "Vishay" V 6600 3950 50  0001 R CNN "Manufacturer"
+F 8 "T7YA474MT20" V 6600 3950 50  0001 R CNN "Manufacturer Part Number"
 	1    6300 3750
 	-1   0    0    1
@@
 F 2 "" H 3850 5600 50  0001 C CNN
 F 3 "~" H 3850 5600 50  0001 C CNN
+F 4 "RS" V 3896 5412 50  0001 R CNN "Supplier"
+F 5 "745-5820" V 3896 5412 50  0001 R CNN "Supplier Part Number"
+F 6 "https://de.rs-online.com/web/p/schiebeschalter/7455820/" V 3896 5412 50  0001 R CNN "Supplier Link"
+F 7 "TE" V 3896 5412 50  0001 R CNN "Manufacturer"
+F 8 "1825163-1" V 3896 5412 50  0001 R CNN "Manufacturer Part Number"
 	1    3850 5600
 	0    -1   -1   0
@@
 F 2 "" H 3850 4800 50  0001 C CNN
 F 3 "~" H 3850 4800 50  0001 C CNN
+F 4 "RS" V 3804 4612 50  0001 R CNN "Supplier"
+F 5 "745-5820" V 3804 4612 50  0001 R CNN "Supplier Part Number"
+F 6 "https://de.rs-online.com/web/p/schiebeschalter/7455820/" V 3804 4612 50  0001 R CNN "Supplier Link"
+F 7 "TE" V 3804 4612 50  0001 R CNN "Manufacturer"
+F 8 "1825163-1" V 3804 4612 50  0001 R CNN "Manufacturer Part Number"
 	2    3850 4800
 	0    -1   1    0

Commit message: Add footprints and part info for IC and inductors
Parts:
- IC1: renamed from U1; value Opamp_Dual_Generic -> TL072; footprint (none) -> Package_DIP:DIP-8_W7.62mm; Manufacturer (none) -> TI; Manufacturer Part Number (none) -> TL072CP; Supplier (none) -> RS; Supplier Link (none) -> https://de.rs-online.com/web/p/operationsverstarker/0304239/; Supplier Part Number (none) -> 304-239
- L1, L2: footprint Inductor_THT:L_Toroid_Horizontal_D17.3mm_P15.24mm_Bourns_2000 -> umidi-wah:Fasel
- SW1: renamed from SW?; value SW_DPDT_x2 -> MMP221; footprint (none) -> umidi-wah:MMP221
Connections:
- net Vref: now also SW1.5 (B); no longer SW1.2 (B)
- net q: now also SW1.2 (B); no longer SW1.5 (B)
- net at L1.1: now also SW1.1 (A); no longer SW1.4 (A)
- net at L1.2: now also SW1.4 (A); no longer SW1.1 (A)
- net at L2.2: now also SW1.6 (C); no longer SW1.3 (C)
- net at L2.1: now also SW1.3 (C); no longer SW1.6 (C)
Changed lines of the file:
@@
 $EndComp
 $Comp
-L Device:Opamp_Dual_Generic U1
+L Device:Opamp_Dual_Generic IC1
 U 1 1 5C8821D1
 P 4200 3200
-F 0 "U1" H 4200 2833 50  0000 C CNN
-F 1 "Opamp_Dual_Generic" H 4200 2924 50  0000 C CNN
-F 2 "" H 4200 3200 50  0001 C CNN
-F 3 "~" H 4200 3200 50  0001 C CNN
+F 0 "IC1" H 4200 2833 50  0000 C CNN
+F 1 "TL072" H 4200 2924 50  0000 C CNN
+F 2 "Package_DIP:DIP-8_W7.62mm" H 4200 3200 50  0001 C CNN
+F 3 "https://docs-emea.rs-online.com/webdocs/1644/0900766b81644f9e.pdf" H 4200 3200 50  0001 C CNN
+F 4 "RS" H 4200 2833 50  0001 C CNN "Supplier"
+F 5 "https://de.rs-online.com/web/p/operationsverstarker/0304239/" H 4200 2833 50  0001 C CNN "Supplier Link"
+F 6 "TI" H 4200 2833 50  0001 C CNN "Manufacturer"
+F 7 "TL072CP" H 4200 2833 50  0001 C CNN "Manufacturer Part Number"
+F 8 "304-239" H 4200 2833 50  0001 C CNN "Supplier Part Number"
 	1    4200 3200
 	1    0    0    1
 $EndComp
 $Comp
-L Device:Opamp_Dual_Generic U1
+L Device:Opamp_Dual_Generic IC1
 U 2 1 5C8824DF
 P 5200 4550
-F 0 "U1" H 5200 4183 50  0000 C CNN
-F 1 "Opamp_Dual_Generic" H 5200 4274 50  0000 C CNN
-F 2 "" H 5200 4550 50  0001 C CNN
-F 3 "~" H 5200 4550 50  0001 C CNN
+F 0 "IC1" H 5200 4183 50  0000 C CNN
+F 1 "TL072" H 5200 4274 50  0000 C CNN
+F 2 "Package_DIP:DIP-8_W7.62mm" H 5200 4550 50  0001 C CNN
+F 3 "https://docs-emea.rs-online.com/webdocs/1644/0900766b81644f9e.pdf" H 5200 4550 50  0001 C CNN
+F 4 "RS" H 5200 4183 50  0001 C CNN "Supplier"
+F 5 "https://de.rs-online.com/web/p/operationsverstarker/0304239/" H 5200 4183 50  0001 C CNN "Supplier Link"
+F 6 "TI" H 5200 4183 50  0001 C CNN "Manufacturer"
+F 7 "TL072CP" H 5200 4183 50  0001 C CNN "Manufacturer Part Number"
+F 8 "304-239" H 5200 4183 50  0001 C CNN "Supplier Part Number"
 	2    5200 4550
 	-1   0    0    1
@@
 F 0 "L1" H 3500 5250 50  0000 L CNN
 F 1 "Fasel Red" H 3350 5150 50  0000 L CNN
-F 2 "Inductor_THT:L_Toroid_Horizontal_D17.3mm_P15.24mm_Bourns_2000" H 3750 5200 50  0001 C CNN
+F 2 "umidi-wah:Fasel" H 3750 5200 50  0001 C CNN
 F 3 "~" H 3750 5200 50  0001 C CNN
 	1    3750 5200
@@
 $EndComp
 $Comp
-L Switch:SW_DPDT_x2 SW?
-U 1 1 5CDB9DAE
+L Switch:SW_DPDT_x2 SW1
+U 2 1 5CDB9DAE
 P 3850 5600
-F 0 "SW?" V 3896 5412 50  0000 R CNN
-F 1 "SW_DPDT_x2" V 3805 5412 50  0000 R CNN
-F 2 "" H 3850 5600 50  0001 C CNN
-F 3 "~" H 3850 5600 50  0001 C CNN
+F 0 "SW1" V 3896 5412 50  0000 R CNN
+F 1 "MMP221" V 3805 5412 50  0000 R CNN
+F 2 "umidi-wah:MMP221" H 3850 5600 50  0001 C CNN
+F 3 "https://docs-emea.rs-online.com/webdocs/0e2b/0900766b80e2b976.pdf" H 3850 5600 50  0001 C CNN
 F 4 "RS" V 3896 5412 50  0001 R CNN "Supplier"
 F 5 "745-5820" V 3896 5412 50  0001 R CNN "Supplier Part Number"
@@
 F 7 "TE" V 3896 5412 50  0001 R CNN "Manufacturer"
 F 8 "1825163-1" V 3896 5412 50  0001 R CNN "Manufacturer Part Number"
-	1    3850 5600
+	2    3850 5600
 	0    -1   -1   0
 $EndComp
 $Comp
-L Switch:SW_DPDT_x2 SW?
-U 2 1 5CDBC60F
+L Switch:SW_DPDT_x2 SW1
+U 1 1 5CDBC60F
 P 3850 4800
-F 0 "SW?" V 3804 4612 50  0000 R CNN
-F 1 "SW_DPDT_x2" V 3895 4612 50  0000 R CNN
-F 2 "" H 3850 4800 50  0001 C CNN
-F 3 "~" H 3850 4800 50  0001 C CNN
+F 0 "SW1" V 3804 4612 50  0000 R CNN
+F 1 "MMP221" V 3895 4612 50  0000 R CNN
+F 2 "umidi-wah:MMP221" H 3850 4800 50  0001 C CNN
+F 3 "https://docs-emea.rs-online.com/webdocs/0e2b/0900766b80e2b976.pdf" H 3850 4800 50  0001 C CNN
 F 4 "RS" V 3804 4612 50  0001 R CNN "Supplier"
 F 5 "745-5820" V 3804 4612 50  0001 R CNN "Supplier Part Number"
@@
 F 7 "TE" V 3804 4612 50  0001 R CNN "Manufacturer"
 F 8 "1825163-1" V 3804 4612 50  0001 R CNN "Manufacturer Part Number"
-	2    3850 4800
+	1    3850 4800
 	0    -1   1    0
 $EndComp
@@
 F 0 "L2" H 4100 5250 50  0000 L CNN
 F 1 "Fasel Yellow" H 4000 5150 50  0000 L CNN
-F 2 "Inductor_THT:L_Toroid_Horizontal_D17.3mm_P15.24mm_Bourns_2000" H 3950 5200 50  0001 C CNN
+F 2 "umidi-wah:Fasel" H 3950 5200 50  0001 C CNN
 F 3 "~" H 3950 5200 50  0001 C CNN
 	1    3950 5200
