File: hardware/led-driver.sch (KiCad schematic (older format))
At the start: 8 parts

Commit message: Edit eval schematic; Import bypass
Parts:
- removed C?: 10uF, symbol Device:C
- R?: value 10k?! -> 1k
Changed lines of the file:
@@
 EESchema Schematic File Version 4
 LIBS:uMIDI-wah-cache
-EELAYER 26 0
+LIBS:bypass-cache
+EELAYER 29 0
 EELAYER END
 $Descr A4 11693 8268
 encoding utf-8
-Sheet 2 2
+Sheet 2 4
 Title ""
 Date ""
@@
 AR Path="/5C8EFAFF/5C8ECBDB" Ref="R?"  Part="1"
 F 0 "R?" V 3493 3100 50  0000 C CNN
-F 1 "10k?!" V 3584 3100 50  0000 C CNN
+F 1 "1k" V 3584 3100 50  0000 C CNN
 F 2 "" V 3630 3100 50  0001 C CNN
 F 3 "~" H 3700 3100 50  0001 C CNN
@@
 $EndComp
 $Comp
-L Device:C C?
-U 1 1 5C8ECE9E
-P 2850 3400
-AR Path="/5C8EC687/5C8ECE9E" Ref="C?"  Part="1"
-AR Path="/5C8EFAFF/5C8ECE9E" Ref="C?"  Part="1"
-F 0 "C?" H 2735 3354 50  0000 R CNN
-F 1 "10uF" H 2735 3445 50  0000 R CNN
-F 2 "" H 2888 3250 50  0001 C CNN
-F 3 "~" H 2850 3400 50  0001 C CNN
-	1    2850 3400
-	-1   0    0    1
-$EndComp
-$Comp
 L Device:L L?
 U 1 1 5C8ECEF6
@@
 	0    -1   -1   0
 $EndComp
-Wire Wire Line
-	2850 3250 2850 3100
 Wire Wire Line
 	3250 3100 3400 3100
@@
 	1    0    0    -1
 $EndComp
-$Comp
-L power:GND #PWR?
-U 1 1 5C8ED241
-P 2850 3700
-AR Path="/5C8EC687/5C8ED241" Ref="#PWR?"  Part="1"
-AR Path="/5C8EFAFF/5C8ED241" Ref="#PWR?"  Part="1"
-F 0 "#PWR?" H 2850 3450 50  0001 C CNN
-F 1 "GND" H 2855 3527 50  0000 C CNN
-F 2 "" H 2850 3700 50  0001 C CNN
-F 3 "" H 2850 3700 50  0001 C CNN
-	1    2850 3700
-	1    0    0    -1
-$EndComp
 Wire Wire Line
 	3400 3550 3400 3700
 Wire Wire Line
-	2850 3550 2850 3700
-Wire Wire Line
-	2850 3100 2950 3100
-Wire Wire Line
-	2650 3100 2850 3100
-Connection ~ 2850 3100
+	2650 3100 2950 3100
 $EndSCHEMATC

Commit message: Annotate schematic
Parts:
- gave numbers to parts that had none: 7
Changed lines of the file:
@@
 $Descr A4 11693 8268
 encoding utf-8
-Sheet 2 4
+Sheet 3 4
 Title ""
 Date ""
@@
 $EndDescr
 $Comp
-L Transistor_BJT:BC547 Q?
+L Transistor_BJT:BC547 Q1
 U 1 1 5C8EC7F4
 P 4150 3100
-AR Path="/5C8EC687/5C8EC7F4" Ref="Q?"  Part="1"
-AR Path="/5C8EFAFF/5C8EC7F4" Ref="Q?"  Part="1"
-F 0 "Q?" H 4341 3146 50  0000 L CNN
+AR Path="/5C8EC687/5C8EC7F4" Ref="Q1"  Part="1"
+AR Path="/5C8EFAFF/5C8EC7F4" Ref="Q2"  Part="1"
+F 0 "Q2" H 4341 3146 50  0000 L CNN
 F 1 "BC547" H 4341 3055 50  0000 L CNN
 F 2 "Package_TO_SOT_THT:TO-92_Inline" H 4350 3025 50  0001 L CIN
@@
 $EndComp
 $Comp
-L Device:LED D?
+L Device:LED D1
 U 1 1 5C8EC98B
 P 4250 2600
-AR Path="/5C8EC687/5C8EC98B" Ref="D?"  Part="1"
-AR Path="/5C8EFAFF/5C8EC98B" Ref="D?"  Part="1"
-F 0 "D?" V 4288 2483 50  0000 R CNN
+AR Path="/5C8EC687/5C8EC98B" Ref="D1"  Part="1"
+AR Path="/5C8EFAFF/5C8EC98B" Ref="D2"  Part="1"
+F 0 "D2" V 4288 2483 50  0000 R CNN
 F 1 "LED" V 4197 2483 50  0000 R CNN
 F 2 "" H 4250 2600 50  0001 C CNN
@@
 	4250 2900 4250 2750
 $Comp
-L power:GND #PWR?
+L power:GND #PWR014
 U 1 1 5C8ECADB
 P 4250 3700
-AR Path="/5C8EC687/5C8ECADB" Ref="#PWR?"  Part="1"
-AR Path="/5C8EFAFF/5C8ECADB" Ref="#PWR?"  Part="1"
-F 0 "#PWR?" H 4250 3450 50  0001 C CNN
+AR Path="/5C8EC687/5C8ECADB" Ref="#PWR014"  Part="1"
+AR Path="/5C8EFAFF/5C8ECADB" Ref="#PWR017"  Part="1"
+F 0 "#PWR017" H 4250 3450 50  0001 C CNN
 F 1 "GND" H 4255 3527 50  0000 C CNN
 F 2 "" H 4250 3700 50  0001 C CNN
@@
 $EndComp
 $Comp
-L Device:R R?
+L Device:R R13
 U 1 1 5C8ECB18
 P 4250 3500
-AR Path="/5C8EC687/5C8ECB18" Ref="R?"  Part="1"
-AR Path="/5C8EFAFF/5C8ECB18" Ref="R?"  Part="1"
-F 0 "R?" H 4320 3546 50  0000 L CNN
+AR Path="/5C8EC687/5C8ECB18" Ref="R13"  Part="1"
+AR Path="/5C8EFAFF/5C8ECB18" Ref="R15"  Part="1"
+F 0 "R15" H 4320 3546 50  0000 L CNN
 F 1 "0" H 4320 3455 50  0000 L CNN
 F 2 "" V 4180 3500 50  0001 C CNN
@@
 	4250 3700 4250 3650
 $Comp
-L Device:R R?
+L Device:R R12
 U 1 1 5C8ECBDB
 P 3700 3100
-AR Path="/5C8EC687/5C8ECBDB" Ref="R?"  Part="1"
-AR Path="/5C8EFAFF/5C8ECBDB" Ref="R?"  Part="1"
-F 0 "R?" V 3493 3100 50  0000 C CNN
+AR Path="/5C8EC687/5C8ECBDB" Ref="R12"  Part="1"
+AR Path="/5C8EFAFF/5C8ECBDB" Ref="R14"  Part="1"
+F 0 "R14" V 3493 3100 50  0000 C CNN
 F 1 "1k" V 3584 3100 50  0000 C CNN
 F 2 "" V 3630 3100 50  0001 C CNN
@@
 	4250 2200 4250 2450
 $Comp
-L Device:C C?
+L Device:C C7
 U 1 1 5C8ECCDD
 P 4500 2200
-AR Path="/5C8EC687/5C8ECCDD" Ref="C?"  Part="1"
-AR Path="/5C8EFAFF/5C8ECCDD" Ref="C?"  Part="1"
-F 0 "C?" V 4248 2200 50  0000 C CNN
+AR Path="/5C8EC687/5C8ECCDD" Ref="C7"  Part="1"
+AR Path="/5C8EFAFF/5C8ECCDD" Ref="C9"  Part="1"
+F 0 "C9" V 4248 2200 50  0000 C CNN
 F 1 "100nF" V 4339 2200 50  0000 C CNN
 F 2 "" H 4538 2050 50  0001 C CNN
@@
 Connection ~ 4250 2200
 $Comp
-L power:GND #PWR?
+L power:GND #PWR015
 U 1 1 5C8ECD89
 P 4750 2300
-AR Path="/5C8EC687/5C8ECD89" Ref="#PWR?"  Part="1"
-AR Path="/5C8EFAFF/5C8ECD89" Ref="#PWR?"  Part="1"
-F 0 "#PWR?" H 4750 2050 50  0001 C CNN
+AR Path="/5C8EC687/5C8ECD89" Ref="#PWR015"  Part="1"
+AR Path="/5C8EFAFF/5C8ECD89" Ref="#PWR018"  Part="1"
+F 0 "#PWR018" H 4750 2050 50  0001 C CNN
 F 1 "GND" H 4755 2127 50  0000 C CNN
 F 2 "" H 4750 2300 50  0001 C CNN
@@
 PWM_Input
 $Comp
-L Device:C C?
+L Device:C C5
 U 1 1 5C8ECE43
 P 3400 3400
-AR Path="/5C8EC687/5C8ECE43" Ref="C?"  Part="1"
-AR Path="/5C8EFAFF/5C8ECE43" Ref="C?"  Part="1"
-F 0 "C?" H 3285 3354 50  0000 R CNN
+AR Path="/5C8EC687/5C8ECE43" Ref="C5"  Part="1"
+AR Path="/5C8EFAFF/5C8ECE43" Ref="C8"  Part="1"
+F 0 "C8" H 3285 3354 50  0000 R CNN
 F 1 "10uF" H 3285 3445 50  0000 R CNN
 F 2 "" H 3438 3250 50  0001 C CNN
@@
 $EndComp
 $Comp
-L Device:L L?
+L Device:L L2
 U 1 1 5C8ECEF6
 P 3100 3100
-AR Path="/5C8EC687/5C8ECEF6" Ref="L?"  Part="1"
-AR Path="/5C8EFAFF/5C8ECEF6" Ref="L?"  Part="1"
-F 0 "L?" V 3290 3100 50  0000 C CNN
+AR Path="/5C8EC687/5C8ECEF6" Ref="L2"  Part="1"
+AR Path="/5C8EFAFF/5C8ECEF6" Ref="L3"  Part="1"
+F 0 "L3" V 3290 3100 50  0000 C CNN
 F 1 "10uH" V 3199 3100 50  0000 C CNN
 F 2 "" H 3100 3100 50  0001 C CNN
@@
 	3400 3100 3550 3100
 $Comp
-L power:GND #PWR?
+L power:GND #PWR013
 U 1 1 5C8ED226
 P 3400 3700
-AR Path="/5C8EC687/5C8ED226" Ref="#PWR?"  Part="1"
-AR Path="/5C8EFAFF/5C8ED226" Ref="#PWR?"  Part="1"
-F 0 "#PWR?" H 3400 3450 50  0001 C CNN
+AR Path="/5C8EC687/5C8ED226" Ref="#PWR013"  Part="1"
+AR Path="/5C8EFAFF/5C8ED226" Ref="#PWR016"  Part="1"
+F 0 "#PWR016" H 3400 3450 50  0001 C CNN
 F 1 "GND" H 3405 3527 50  0000 C CNN
 F 2 "" H 3400 3700 50  0001 C CNN

Commit message: Use 0805 footprint for all resistors
Parts:
- R12, R13: footprint (none) -> Resistors_SMD:R_0805
Changed lines of the file:
@@
 F 0 "R15" H 4320 3546 50  0000 L CNN
 F 1 "0" H 4320 3455 50  0000 L CNN
-F 2 "" V 4180 3500 50  0001 C CNN
-F 3 "~" H 4250 3500 50  0001 C CNN
+F 2 "Resistors_SMD:R_0805" V 4180 3500 50  0001 C CNN
+F 3 "" H 4250 3500 50  0001 C CNN
 	1    4250 3500
 	1    0    0    -1
@@
 F 0 "R14" V 3493 3100 50  0000 C CNN
 F 1 "1k" V 3584 3100 50  0000 C CNN
-F 2 "" V 3630 3100 50  0001 C CNN
-F 3 "~" H 3700 3100 50  0001 C CNN
+F 2 "Resistors_SMD:R_0805" V 3630 3100 50  0001 C CNN
+F 3 "" H 3700 3100 50  0001 C CNN
 	1    3700 3100
 	0    1    1    0

Commit message: Use 0805 footprint for all capacitors
Parts:
- C5, C7: footprint (none) -> Capacitors_SMD:C_0805
Changed lines of the file:
@@
 F 0 "C9" V 4248 2200 50  0000 C CNN
 F 1 "100nF" V 4339 2200 50  0000 C CNN
-F 2 "" H 4538 2050 50  0001 C CNN
-F 3 "~" H 4500 2200 50  0001 C CNN
+F 2 "Capacitors_SMD:C_0805" H 4538 2050 50  0001 C CNN
+F 3 "" H 4500 2200 50  0001 C CNN
 	1    4500 2200
 	0    1    1    0
@@
 F 0 "C8" H 3285 3354 50  0000 R CNN
 F 1 "10uF" H 3285 3445 50  0000 R CNN
-F 2 "" H 3438 3250 50  0001 C CNN
-F 3 "~" H 3400 3400 50  0001 C CNN
+F 2 "Capacitors_SMD:C_0805" H 3438 3250 50  0001 C CNN
+F 3 "" H 3400 3400 50  0001 C CNN
 	1    3400 3400
 	-1   0    0    1

Commit message: Add footprints and part info for IC and inductors
Parts:
- renumbered L2 to L4
Changed lines of the file:
@@
 $Descr A4 11693 8268
 encoding utf-8
-Sheet 3 4
+Sheet 2 4
 Title ""
 Date ""
@@
 AR Path="/5C8EC687/5C8EC7F4" Ref="Q1"  Part="1"
 AR Path="/5C8EFAFF/5C8EC7F4" Ref="Q2"  Part="1"
-F 0 "Q2" H 4341 3146 50  0000 L CNN
+F 0 "Q1" H 4341 3146 50  0000 L CNN
 F 1 "BC547" H 4341 3055 50  0000 L CNN
 F 2 "Package_TO_SOT_THT:TO-92_Inline" H 4350 3025 50  0001 L CIN
@@
 AR Path="/5C8EC687/5C8EC98B" Ref="D1"  Part="1"
 AR Path="/5C8EFAFF/5C8EC98B" Ref="D2"  Part="1"
-F 0 "D2" V 4288 2483 50  0000 R CNN
+F 0 "D1" V 4288 2483 50  0000 R CNN
 F 1 "LED" V 4197 2483 50  0000 R CNN
 F 2 "" H 4250 2600 50  0001 C CNN
@@
 AR Path="/5C8EC687/5C8ECADB" Ref="#PWR014"  Part="1"
 AR Path="/5C8EFAFF/5C8ECADB" Ref="#PWR017"  Part="1"
-F 0 "#PWR017" H 4250 3450 50  0001 C CNN
+F 0 "#PWR014" H 4250 3450 50  0001 C CNN
 F 1 "GND" H 4255 3527 50  0000 C CNN
 F 2 "" H 4250 3700 50  0001 C CNN
@@
 AR Path="/5C8EC687/5C8ECB18" Ref="R13"  Part="1"
 AR Path="/5C8EFAFF/5C8ECB18" Ref="R15"  Part="1"
-F 0 "R15" H 4320 3546 50  0000 L CNN
+F 0 "R13" H 4320 3546 50  0000 L CNN
 F 1 "0" H 4320 3455 50  0000 L CNN
 F 2 "Resistors_SMD:R_0805" V 4180 3500 50  0001 C CNN
@@
 AR Path="/5C8EC687/5C8ECBDB" Ref="R12"  Part="1"
 AR Path="/5C8EFAFF/5C8ECBDB" Ref="R14"  Part="1"
-F 0 "R14" V 3493 3100 50  0000 C CNN
+F 0 "R12" V 3493 3100 50  0000 C CNN
 F 1 "1k" V 3584 3100 50  0000 C CNN
 F 2 "Resistors_SMD:R_0805" V 3630 3100 50  0001 C CNN
@@
 AR Path="/5C8EC687/5C8ECCDD" Ref="C7"  Part="1"
 AR Path="/5C8EFAFF/5C8ECCDD" Ref="C9"  Part="1"
-F 0 "C9" V 4248 2200 50  0000 C CNN
+F 0 "C7" V 4248 2200 50  0000 C CNN
 F 1 "100nF" V 4339 2200 50  0000 C CNN
 F 2 "Capacitors_SMD:C_0805" H 4538 2050 50  0001 C CNN
@@
 AR Path="/5C8EC687/5C8ECD89" Ref="#PWR015"  Part="1"
 AR Path="/5C8EFAFF/5C8ECD89" Ref="#PWR018"  Part="1"
-F 0 "#PWR018" H 4750 2050 50  0001 C CNN
+F 0 "#PWR015" H 4750 2050 50  0001 C CNN
 F 1 "GND" H 4755 2127 50  0000 C CNN
 F 2 "" H 4750 2300 50  0001 C CNN
@@
 AR Path="/5C8EC687/5C8ECE43" Ref="C5"  Part="1"
 AR Path="/5C8EFAFF/5C8ECE43" Ref="C8"  Part="1"
-F 0 "C8" H 3285 3354 50  0000 R CNN
+F 0 "C5" H 3285 3354 50  0000 R CNN
 F 1 "10uF" H 3285 3445 50  0000 R CNN
 F 2 "Capacitors_SMD:C_0805" H 3438 3250 50  0001 C CNN
@@
 $EndComp
 $Comp
-L Device:L L2
+L Device:L L4
 U 1 1 5C8ECEF6
 P 3100 3100
-AR Path="/5C8EC687/5C8ECEF6" Ref="L2"  Part="1"
+AR Path="/5C8EC687/5C8ECEF6" Ref="L4"  Part="1"
 AR Path="/5C8EFAFF/5C8ECEF6" Ref="L3"  Part="1"
-F 0 "L3" V 3290 3100 50  0000 C CNN
+F 0 "L4" V 3290 3100 50  0000 C CNN
 F 1 "10uH" V 3199 3100 50  0000 C CNN
 F 2 "" H 3100 3100 50  0001 C CNN
@@
 AR Path="/5C8EC687/5C8ED226" Ref="#PWR013"  Part="1"
 AR Path="/5C8EFAFF/5C8ED226" Ref="#PWR016"  Part="1"
-F 0 "#PWR016" H 3400 3450 50  0001 C CNN
+F 0 "#PWR013" H 3400 3450 50  0001 C CNN
 F 1 "GND" H 3405 3527 50  0000 C CNN
 F 2 "" H 3400 3700 50  0001 C CNN

Commit message: Select and update LED circuit
Parts:
- added D5: LED, LED_SMD:LED_0805_2012Metric, symbol Device:LED
- added R23: 1k, Resistors_SMD:R_0805, symbol Device:R
- D1: footprint (none) -> LED_SMD:LED_0805_2012Metric; Manufacturer (none) -> ROHM; Manufacturer Part Number (none) -> SML-210PTT86; Supplier (none) -> RS; Supplier Link (none) -> https://de.rs-online.com/web/p/leds-sichtbares-licht/700789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; Supplier Part Number (none) -> 700-7890
Connections:
- net Led_Supply: now also R23.2; no longer D1.2 (A)
- new net: D1.2 (A), D5.1 (K)
- new net: D5.2 (A), R23.1
Other:
- moved on the sheet: C9
Changed lines of the file:
@@
 AR Path="/5C8EC687/5C8EC7F4" Ref="Q1"  Part="1"
 AR Path="/5C8EFAFF/5C8EC7F4" Ref="Q2"  Part="1"
-F 0 "Q1" H 4341 3146 50  0000 L CNN
+F 0 "Q2" H 4341 3146 50  0000 L CNN
 F 1 "BC547" H 4341 3055 50  0000 L CNN
 F 2 "Package_TO_SOT_THT:TO-92_Inline" H 4350 3025 50  0001 L CIN
@@
 AR Path="/5C8EC687/5C8EC98B" Ref="D1"  Part="1"
 AR Path="/5C8EFAFF/5C8EC98B" Ref="D2"  Part="1"
-F 0 "D1" V 4288 2483 50  0000 R CNN
+F 0 "D2" V 4288 2483 50  0000 R CNN
 F 1 "LED" V 4197 2483 50  0000 R CNN
-F 2 "" H 4250 2600 50  0001 C CNN
-F 3 "~" H 4250 2600 50  0001 C CNN
+F 2 "LED_SMD:LED_0805_2012Metric" H 4250 2600 50  0001 C CNN
+F 3 "http://datasheet.octopart.com/SML-210PTT86-Rohm-datasheet-12523978.pdf" H 4250 2600 50  0001 C CNN
+F 4 "RS" V 4288 2483 50  0001 R CNN "Supplier"
+F 5 "700-7890" V 4288 2483 50  0001 R CNN "Supplier Part Number"
+F 6 "https://de.rs-online.com/web/p/leds-sichtbares-licht/7007890/" V 4288 2483 50  0001 R CNN "Supplier Link"
+F 7 "ROHM" V 4288 2483 50  0001 R CNN "Manufacturer"
+F 8 "SML-210PTT86" V 4288 2483 50  0001 R CNN "Manufacturer Part Number"
 	1    4250 2600
 	0    -1   -1   0
@@
 AR Path="/5C8EC687/5C8ECB18" Ref="R13"  Part="1"
 AR Path="/5C8EFAFF/5C8ECB18" Ref="R15"  Part="1"
-F 0 "R13" H 4320 3546 50  0000 L CNN
+F 0 "R15" H 4320 3546 50  0000 L CNN
 F 1 "0" H 4320 3455 50  0000 L CNN
 F 2 "Resistors_SMD:R_0805" V 4180 3500 50  0001 C CNN
@@
 AR Path="/5C8EC687/5C8ECBDB" Ref="R12"  Part="1"
 AR Path="/5C8EFAFF/5C8ECBDB" Ref="R14"  Part="1"
-F 0 "R12" V 3493 3100 50  0000 C CNN
+F 0 "R14" V 3493 3100 50  0000 C CNN
 F 1 "1k" V 3584 3100 50  0000 C CNN
 F 2 "Resistors_SMD:R_0805" V 3630 3100 50  0001 C CNN
@@
 Wire Wire Line
 	3850 3100 3950 3100
-Text HLabel 4050 2200 0    50   Input ~ 0
+Text HLabel 4050 1400 0    50   Input ~ 0
 Led_Supply
 Wire Wire Line
-	4050 2200 4250 2200
-Wire Wire Line
-	4250 2200 4250 2450
+	4050 1400 4250 1400
+Wire Wire Line
+	4250 1400 4250 1650
 $Comp
 L Device:C C7
 U 1 1 5C8ECCDD
-P 4500 2200
+P 4500 1400
 AR Path="/5C8EC687/5C8ECCDD" Ref="C7"  Part="1"
 AR Path="/5C8EFAFF/5C8ECCDD" Ref="C9"  Part="1"
-F 0 "C7" V 4248 2200 50  0000 C CNN
-F 1 "100nF" V 4339 2200 50  0000 C CNN
-F 2 "Capacitors_SMD:C_0805" H 4538 2050 50  0001 C CNN
-F 3 "" H 4500 2200 50  0001 C CNN
-	1    4500 2200
+F 0 "C9" V 4248 1400 50  0000 C CNN
+F 1 "100nF" V 4339 1400 50  0000 C CNN
+F 2 "Capacitors_SMD:C_0805" H 4538 1250 50  0001 C CNN
+F 3 "" H 4500 1400 50  0001 C CNN
+	1    4500 1400
 	0    1    1    0
 $EndComp
 Wire Wire Line
-	4350 2200 4250 2200
-Connection ~ 4250 2200
+	4350 1400 4250 1400
+Connection ~ 4250 1400
 $Comp
 L power:GND #PWR015
 U 1 1 5C8ECD89
-P 4750 2300
+P 4750 1500
 AR Path="/5C8EC687/5C8ECD89" Ref="#PWR015"  Part="1"
 AR Path="/5C8EFAFF/5C8ECD89" Ref="#PWR018"  Part="1"
-F 0 "#PWR018" H 4750 2050 50  0001 C CNN
-F 1 "GND" H 4755 2127 50  0000 C CNN
-F 2 "" H 4750 2300 50  0001 C CNN
-F 3 "" H 4750 2300 50  0001 C CNN
-	1    4750 2300
-	1    0    0    -1
-$EndComp
-Wire Wire Line
-	4750 2300 4750 2200
-Wire Wire Line
-	4750 2200 4650 2200
+F 0 "#PWR018" H 4750 1250 50  0001 C CNN
+F 1 "GND" H 4755 1327 50  0000 C CNN
+F 2 "" H 4750 1500 50  0001 C CNN
+F 3 "" H 4750 1500 50  0001 C CNN
+	1    4750 1500
+	1    0    0    -1
+$EndComp
+Wire Wire Line
+	4750 1500 4750 1400
+Wire Wire Line
+	4750 1400 4650 1400
 Text HLabel 2650 3100 0    50   Input ~ 0
 PWM_Input
@@
 AR Path="/5C8EC687/5C8ECE43" Ref="C5"  Part="1"
 AR Path="/5C8EFAFF/5C8ECE43" Ref="C8"  Part="1"
-F 0 "C5" H 3285 3354 50  0000 R CNN
+F 0 "C8" H 3285 3354 50  0000 R CNN
 F 1 "10uF" H 3285 3445 50  0000 R CNN
 F 2 "Capacitors_SMD:C_0805" H 3438 3250 50  0001 C CNN
@@
 AR Path="/5C8EC687/5C8ECEF6" Ref="L4"  Part="1"
 AR Path="/5C8EFAFF/5C8ECEF6" Ref="L3"  Part="1"
-F 0 "L4" V 3290 3100 50  0000 C CNN
+F 0 "L3" V 3290 3100 50  0000 C CNN
 F 1 "10uH" V 3199 3100 50  0000 C CNN
 F 2 "" H 3100 3100 50  0001 C CNN
@@
 Wire Wire Line
 	2650 3100 2950 3100
+$Comp
+L Device:LED D5
+U 1 1 5CD989FA
+P 4250 2200
+AR Path="/5C8EC687/5CD989FA" Ref="D5"  Part="1"
+AR Path="/5C8EFAFF/5CD989FA" Ref="D6"  Part="1"
+F 0 "D6" V 4288 2083 50  0000 R CNN
+F 1 "LED" V 4197 2083 50  0000 R CNN
+F 2 "LED_SMD:LED_0805_2012Metric" H 4250 2200 50  0001 C CNN
+F 3 "http://datasheet.octopart.com/SML-210PTT86-Rohm-datasheet-12523978.pdf" H 4250 2200 50  0001 C CNN
+F 4 "RS" V 4288 2083 50  0001 R CNN "Supplier"
+F 5 "700-7890" V 4288 2083 50  0001 R CNN "Supplier Part Number"
+F 6 "https://de.rs-online.com/web/p/leds-sichtbares-licht/7007890/" V 4288 2083 50  0001 R CNN "Supplier Link"
+F 7 "ROHM" V 4288 2083 50  0001 R CNN "Manufacturer"
+F 8 "SML-210PTT86" V 4288 2083 50  0001 R CNN "Manufacturer Part Number"
+	1    4250 2200
+	0    -1   -1   0
+$EndComp
+$Comp
+L Device:R R23
+U 1 1 5CD998D9
+P 4250 1800
+AR Path="/5C8EC687/5CD998D9" Ref="R23"  Part="1"
+AR Path="/5C8EFAFF/5CD998D9" Ref="R24"  Part="1"
+F 0 "R24" V 4043 1800 50  0000 C CNN
+F 1 "1k" V 4134 1800 50  0000 C CNN
+F 2 "Resistors_SMD:R_0805" V 4180 1800 50  0001 C CNN
+F 3 "" H 4250 1800 50  0001 C CNN
+	1    4250 1800
+	-1   0    0    1
+$EndComp
+Wire Wire Line
+	4250 1950 4250 2050
+Wire Wire Line
+	4250 2350 4250 2450
 $EndSCHEMATC
