File: hardware/bypass.sch (KiCad schematic (older format))
At the start: 10 parts, among them Q1 BSS138

Commit message: Annotate schematic
Changed lines of the file:
@@
 AR Path="/56223A6E/54E9BE9F/54D79A29" Ref="REL5"  Part="1"
 AR Path="/56223A7C/54E9BE9F/54D79A29" Ref="REL6"  Part="1"
-AR Path="/5CD91DFE/54D79A29" Ref="REL?"  Part="1"
-F 0 "REL?" H 8050 3500 60  0000 C CNN
+AR Path="/5CD91DFE/54D79A29" Ref="REL1"  Part="1"
+F 0 "REL1" H 8050 3500 60  0000 C CNN
 F 1 "Omron G6K-2P-5VCD" H 8050 3600 60  0000 C CNN
 F 2 "uMIDI-switcher:Omron_G6K-2P" H 8050 3300 60  0001 C CNN
@@
 AR Path="/56223A6E/54E9BE9F/54D79A79" Ref="REL5"  Part="2"
 AR Path="/56223A7C/54E9BE9F/54D79A79" Ref="REL6"  Part="2"
-AR Path="/5CD91DFE/54D79A79" Ref="REL?"  Part="2"
-F 0 "REL?" H 3700 4000 60  0000 C CNN
+AR Path="/5CD91DFE/54D79A79" Ref="REL1"  Part="2"
+F 0 "REL1" H 3700 4000 60  0000 C CNN
 F 1 "Omron G6K-2P-5VCD" H 3700 3500 60  0001 C CNN
 F 2 "uMIDI-switcher:Omron_G6K-2P" H 3700 3800 60  0001 C CNN
@@
 AR Path="/56223A6E/54E9BE9F/54D79AAA" Ref="REL5"  Part="3"
 AR Path="/56223A7C/54E9BE9F/54D79AAA" Ref="REL6"  Part="3"
-AR Path="/5CD91DFE/54D79AAA" Ref="REL?"  Part="3"
-F 0 "REL?" H 5200 4000 60  0000 C CNN
+AR Path="/5CD91DFE/54D79AAA" Ref="REL1"  Part="3"
+F 0 "REL1" H 5200 4000 60  0000 C CNN
 F 1 "Omron G6K-2P-5VCD" H 4850 4150 60  0001 C CNN
 F 2 "uMIDI-switcher:Omron_G6K-2P" H 5200 3800 60  0001 C CNN
@@
 AR Path="/56223A7C/54E9BE9F/54D79DA0" Ref="R22"  Part="1"
 AR Path="/56223A90/54E9BE9F/54D79DA0" Ref="R27"  Part="1"
-AR Path="/5CD91DFE/54D79DA0" Ref="R?"  Part="1"
-F 0 "R?" V 4100 4150 50  0000 C CNN
+AR Path="/5CD91DFE/54D79DA0" Ref="R16"  Part="1"
+F 0 "R16" V 4100 4150 50  0000 C CNN
 F 1 "100M" V 4200 4150 50  0000 C CNN
 F 2 "Resistors_SMD:R_0603" V 4130 4150 30  0001 C CNN
@@
 AR Path="/56223A7C/54E9BE9F/54D7A6A7" Ref="D6"  Part="1"
 AR Path="/56223A90/54E9BE9F/54D7A6A7" Ref="D7"  Part="1"
-AR Path="/5CD91DFE/54D7A6A7" Ref="D?"  Part="1"
-F 0 "D?" H 7750 3400 50  0000 C CNN
+AR Path="/5CD91DFE/54D7A6A7" Ref="D3"  Part="1"
+F 0 "D3" H 7750 3400 50  0000 C CNN
 F 1 "1N4148" H 7750 3200 50  0000 C CNN
 F 2 "Diodes_SMD:SOD-123" H 7750 3300 60  0001 C CNN
@@
 AR Path="/56223A7C/54E9BE9F/54D7A960" Ref="#PWR065"  Part="1"
 AR Path="/56223A90/54E9BE9F/54D7A960" Ref="#PWR072"  Part="1"
-AR Path="/5CD91DFE/54D7A960" Ref="#PWR?"  Part="1"
-F 0 "#PWR?" H 7900 4550 60  0001 C CNN
+AR Path="/5CD91DFE/54D7A960" Ref="#PWR024"  Part="1"
+F 0 "#PWR024" H 7900 4550 60  0001 C CNN
 F 1 "GND" H 7900 4650 60  0000 C CNN
 F 2 "" H 7900 4800 60  0000 C CNN
@@
 AR Path="/56223A7C/54E9BE9F/54D7AAB4" Ref="C21"  Part="1"
 AR Path="/56223A90/54E9BE9F/54D7AAB4" Ref="C23"  Part="1"
-AR Path="/5CD91DFE/54D7AAB4" Ref="C?"  Part="1"
-F 0 "C?" H 6650 3350 50  0000 L CNN
+AR Path="/5CD91DFE/54D7AAB4" Ref="C10"  Part="1"
+F 0 "C10" H 6650 3350 50  0000 L CNN
 F 1 "100n" H 6650 3150 50  0000 L CNN
 F 2 "Capacitors_SMD:C_0603" H 6638 3100 30  0001 C CNN
@@
 AR Path="/56223A7C/54E9BE9F/54D7AB88" Ref="#PWR066"  Part="1"
 AR Path="/56223A90/54E9BE9F/54D7AB88" Ref="#PWR073"  Part="1"
-AR Path="/5CD91DFE/54D7AB88" Ref="#PWR?"  Part="1"
-F 0 "#PWR?" H 6600 3200 60  0001 C CNN
+AR Path="/5CD91DFE/54D7AB88" Ref="#PWR021"  Part="1"
+F 0 "#PWR021" H 6600 3200 60  0001 C CNN
 F 1 "GND" H 6600 3300 60  0000 C CNN
 F 2 "" H 6600 3450 60  0000 C CNN
@@
 AR Path="/56223A7C/54E9BE9F/54D7ADF3" Ref="R26"  Part="1"
 AR Path="/56223A90/54E9BE9F/54D7ADF3" Ref="R31"  Part="1"
-AR Path="/5CD91DFE/54D7ADF3" Ref="R?"  Part="1"
-F 0 "R?" V 7580 4600 50  0000 C CNN
+AR Path="/5CD91DFE/54D7ADF3" Ref="R20"  Part="1"
+F 0 "R20" V 7580 4600 50  0000 C CNN
 F 1 "10k" V 7507 4601 50  0000 C CNN
 F 2 "Resistors_SMD:R_0603" V 7430 4600 30  0001 C CNN
@@
 AR Path="/56223A90/54E9BE9F/54D7AECB" Ref="Q6"  Part="1"
 AR Path="/54D7AECB" Ref="Q1"  Part="1"
-AR Path="/5CD91DFE/54D7AECB" Ref="Q?"  Part="1"
-F 0 "Q?" H 7800 4101 40  0000 R CNN
+AR Path="/5CD91DFE/54D7AECB" Ref="Q3"  Part="1"
+F 0 "Q3" H 7800 4101 40  0000 R CNN
 F 1 "BSS138" H 7800 4400 40  0000 R CNN
 F 2 "Housings_SOT-23_SOT-143_TSOT-6:SOT-23" H 7670 4352 29  0001 C CNN
@@
 AR Path="/56223A7C/54E9BE9F/54D7B0C5" Ref="#PWR067"  Part="1"
 AR Path="/56223A90/54E9BE9F/54D7B0C5" Ref="#PWR074"  Part="1"
-AR Path="/5CD91DFE/54D7B0C5" Ref="#PWR?"  Part="1"
-F 0 "#PWR?" H 7500 4550 60  0001 C CNN
+AR Path="/5CD91DFE/54D7B0C5" Ref="#PWR023"  Part="1"
+F 0 "#PWR023" H 7500 4550 60  0001 C CNN
 F 1 "GND" H 7500 4650 60  0000 C CNN
 F 2 "" H 7500 4800 60  0000 C CNN
@@
 AR Path="/56223A7C/54E9BE9F/54D7C711" Ref="R25"  Part="1"
 AR Path="/56223A90/54E9BE9F/54D7C711" Ref="R30"  Part="1"
-AR Path="/5CD91DFE/54D7C711" Ref="R?"  Part="1"
-F 0 "R?" V 6850 3000 50  0000 C CNN
+AR Path="/5CD91DFE/54D7C711" Ref="R19"  Part="1"
+F 0 "R19" V 6850 3000 50  0000 C CNN
 F 1 "180" V 6957 3001 50  0000 C CNN
 F 2 "Resistors_SMD:R_0603" V 6880 3000 30  0001 C CNN
@@
 AR Path="/56223A7C/54E9BE9F/54D7C874" Ref="C22"  Part="1"
 AR Path="/56223A90/54E9BE9F/54D7C874" Ref="C24"  Part="1"
-AR Path="/5CD91DFE/54D7C874" Ref="C?"  Part="1"
-F 0 "C?" H 7350 3350 50  0000 L CNN
+AR Path="/5CD91DFE/54D7C874" Ref="C11"  Part="1"
+F 0 "C11" H 7350 3350 50  0000 L CNN
 F 1 "100n" H 7350 3150 50  0000 L CNN
 F 2 "Capacitors_SMD:C_0603" H 7338 3100 30  0001 C CNN
@@
 AR Path="/56223A7C/54E9BE9F/54D7C87A" Ref="#PWR068"  Part="1"
 AR Path="/56223A90/54E9BE9F/54D7C87A" Ref="#PWR075"  Part="1"
-AR Path="/5CD91DFE/54D7C87A" Ref="#PWR?"  Part="1"
-F 0 "#PWR?" H 7300 3200 60  0001 C CNN
+AR Path="/5CD91DFE/54D7C87A" Ref="#PWR022"  Part="1"
+F 0 "#PWR022" H 7300 3200 60  0001 C CNN
 F 1 "GND" H 7300 3300 60  0000 C CNN
 F 2 "" H 7300 3450 60  0000 C CNN
@@
 AR Path="/56223A7C/54E9BE9F/54EA1C00" Ref="#PWR069"  Part="1"
 AR Path="/56223A90/54E9BE9F/54EA1C00" Ref="#PWR076"  Part="1"
-AR Path="/5CD91DFE/54EA1C00" Ref="#PWR?"  Part="1"
-F 0 "#PWR?" H 4450 4250 60  0001 C CNN
+AR Path="/5CD91DFE/54EA1C00" Ref="#PWR019"  Part="1"
+F 0 "#PWR019" H 4450 4250 60  0001 C CNN
 F 1 "GNDA" H 4450 4350 60  0000 C CNN
 F 2 "" H 4450 4500 60  0000 C CNN
@@
 AR Path="/56223A7C/54E9BE9F/54E940D4" Ref="#PWR070"  Part="1"
 AR Path="/56223A90/54E9BE9F/54E940D4" Ref="#PWR077"  Part="1"
-AR Path="/5CD91DFE/54E940D4" Ref="#PWR?"  Part="1"
-F 0 "#PWR?" H 6350 2800 60  0001 C CNN
+AR Path="/5CD91DFE/54E940D4" Ref="#PWR020"  Part="1"
+F 0 "#PWR020" H 6350 2800 60  0001 C CNN
 F 1 "+9V" H 6350 3090 60  0000 C CNN
 F 2 "" H 6350 2950 60  0000 C CNN
@@
 AR Path="/56223A7C/54E9BE9F/55F44BB0" Ref="R23"  Part="1"
 AR Path="/56223A90/54E9BE9F/55F44BB0" Ref="R28"  Part="1"
-AR Path="/5CD91DFE/55F44BB0" Ref="R?"  Part="1"
-F 0 "R?" V 4350 4150 50  0000 C CNN
+AR Path="/5CD91DFE/55F44BB0" Ref="R17"  Part="1"
+F 0 "R17" V 4350 4150 50  0000 C CNN
 F 1 "100M" V 4450 4150 50  0000 C CNN
 F 2 "Resistors_SMD:R_0603" V 4380 4150 30  0001 C CNN
@@
 AR Path="/56223A7C/54E9BE9F/55F44BF3" Ref="R24"  Part="1"
 AR Path="/56223A90/54E9BE9F/55F44BF3" Ref="R29"  Part="1"
-AR Path="/5CD91DFE/55F44BF3" Ref="R?"  Part="1"
-F 0 "R?" V 4600 4150 50  0000 C CNN
+AR Path="/5CD91DFE/55F44BF3" Ref="R18"  Part="1"
+F 0 "R18" V 4600 4150 50  0000 C CNN
 F 1 "100M" V 4700 4150 50  0000 C CNN
 F 2 "Resistors_SMD:R_0603" V 4630 4150 30  0001 C CNN

Commit message: Use 0805 footprint for all resistors
Parts:
- R2: footprint Resistors_SMD:R_0603 -> Resistors_SMD:R_0805; Manufacturer Vishay/Dale -> (none); Manufacturer Link http://www.vishay.com/resistors-fixed/list/product-20011/ -> (none); Manufacturer Part Number CRCW0603100MJPEAHR -> (none); Supplier Mouser -> (none); Supplier Link http://eu.mouser.com/ProductDetail/Vishay-Dale/CRCW0603100M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 -> (none); Supplier Part Number 71-CRCW0603100MJPEA -> (none)
- R3, R4, R5, R6: footprint Resistors_SMD:R_0603 -> Resistors_SMD:R_0805
Changed lines of the file:
@@
 F 0 "R16" V 4100 4150 50  0000 C CNN
 F 1 "100M" V 4200 4150 50  0000 C CNN
-F 2 "Resistors_SMD:R_0603" V 4130 4150 30  0001 C CNN
-F 3 "http://www.vishay.com/docs/20022/dcrcwhe3.pdf" H 4100 4150 60  0001 C CNN
-F 4 "Mouser" H 4100 4150 60  0001 C CNN "Supplier"
-F 5 "71-CRCW0603100MJPEA" H 4100 4150 60  0001 C CNN "Supplier Part Number"
-F 6 "http://eu.mouser.com/ProductDetail/Vishay-Dale/CRCW0603100MJPEAHR/?qs=sGAEpiMZZMu61qfTUdNhGwALI1ohWcNj4pxTQEkdYlc%3d" H 4100 4150 60  0001 C CNN "Supplier Link"
-F 7 "Vishay/Dale" H 4100 4150 60  0001 C CNN "Manufacturer"
-F 8 "CRCW0603100MJPEAHR" H 4100 4150 60  0001 C CNN "Manufacturer Part Number"
-F 9 "http://www.vishay.com/resistors-fixed/list/product-20011/" H 4100 4150 60  0001 C CNN "Manufacturer Link"
+F 2 "Resistors_SMD:R_0805" V 4130 4150 30  0001 C CNN
+F 3 "" H 4100 4150 60  0001 C CNN
 	1    4200 4150
 	1    0    0    -1
@@
 F 0 "R20" V 7580 4600 50  0000 C CNN
 F 1 "10k" V 7507 4601 50  0000 C CNN
-F 2 "Resistors_SMD:R_0603" V 7430 4600 30  0001 C CNN
-F 3 "http://www.vishay.com/docs/20022/dcrcwhe3.pdf" H 7580 4600 60  0001 C CNN
+F 2 "Resistors_SMD:R_0805" V 7430 4600 30  0001 C CNN
+F 3 "" H 7580 4600 60  0001 C CNN
 F 4 "Mouser" H 7580 4600 60  0001 C CNN "Supplier"
 F 5 "71-CRCW0603J-10K-E3" H 7580 4600 60  0001 C CNN "Supplier Part Number"
@@
 F 0 "R19" V 6850 3000 50  0000 C CNN
 F 1 "180" V 6957 3001 50  0000 C CNN
-F 2 "Resistors_SMD:R_0603" V 6880 3000 30  0001 C CNN
-F 3 "http://www.vishay.com/docs/20022/dcrcwhe3.pdf" H 6850 3000 60  0001 C CNN
+F 2 "Resistors_SMD:R_0805" V 6880 3000 30  0001 C CNN
+F 3 "" H 6850 3000 60  0001 C CNN
 F 4 "Mouser" H 6850 3000 60  0001 C CNN "Supplier"
 F 5 "71-CRCW0603J-180-E3 " H 6850 3000 60  0001 C CNN "Supplier Part Number"
@@
 F 0 "R17" V 4350 4150 50  0000 C CNN
 F 1 "100M" V 4450 4150 50  0000 C CNN
-F 2 "Resistors_SMD:R_0603" V 4380 4150 30  0001 C CNN
-F 3 "http://www.vishay.com/docs/20022/dcrcwhe3.pdf" H 4350 4150 60  0001 C CNN
+F 2 "Resistors_SMD:R_0805" V 4380 4150 30  0001 C CNN
+F 3 "" H 4350 4150 60  0001 C CNN
 F 4 "Mouser" H 4350 4150 60  0001 C CNN "Supplier"
 F 5 "71-CRCW0603100MJPEA" H 4350 4150 60  0001 C CNN "Supplier Part Number"
@@
 F 0 "R18" V 4600 4150 50  0000 C CNN
 F 1 "100M" V 4700 4150 50  0000 C CNN
-F 2 "Resistors_SMD:R_0603" V 4630 4150 30  0001 C CNN
-F 3 "http://www.vishay.com/docs/20022/dcrcwhe3.pdf" H 4600 4150 60  0001 C CNN
+F 2 "Resistors_SMD:R_0805" V 4630 4150 30  0001 C CNN
+F 3 "" H 4600 4150 60  0001 C CNN
 F 4 "Mouser" H 4600 4150 60  0001 C CNN "Supplier"
 F 5 "71-CRCW0603100MJPEA" H 4600 4150 60  0001 C CNN "Supplier Part Number"

Commit message: Use 0805 footprint for all capacitors
Parts:
- C13: footprint Capacitors_SMD:C_0603 -> Capacitors_SMD:C_0805; Manufacturer Murata -> (none); Manufacturer Part Number GRM188R71E104KA01D -> (none); Supplier Mouser -> (none); Supplier Link http://eu.mouser.com/ProductDetail/Murata-Electronics/GRM18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 -> (none); Supplier Part Number 81-GRM39X104K25 -> (none)
- C14: footprint Capacitors_SMD:C_0603 -> Capacitors_SMD:C_0805
Changed lines of the file:
@@
 F 0 "C10" H 6650 3350 50  0000 L CNN
 F 1 "100n" H 6650 3150 50  0000 L CNN
-F 2 "Capacitors_SMD:C_0603" H 6638 3100 30  0001 C CNN
-F 3 "http://psearch.en.murata.com/capacitor/product/GRM188R71E104KA01%23.pdf" H 6650 3350 60  0001 C CNN
-F 4 "Mouser" H 3650 5050 60  0001 C CNN "Supplier"
-F 5 "81-GRM39X104K25 " H 3650 5050 60  0001 C CNN "Supplier Part Number"
-F 6 "http://eu.mouser.com/ProductDetail/Murata-Electronics/GRM188R71E104KA01D/?qs=sGAEpiMZZMs0AnBnWHyRQNOmsPzkISN0CS9R%252buxD0A8%3d" H 3650 5050 60  0001 C CNN "Supplier Link"
-F 7 "Murata" H 3650 5050 60  0001 C CNN "Manufacturer"
-F 8 "GRM188R71E104KA01D" H 3650 5050 60  0001 C CNN "Manufacturer Part Number"
+F 2 "Capacitors_SMD:C_0805" H 6638 3100 30  0001 C CNN
+F 3 "" H 6650 3350 60  0001 C CNN
 	1    6600 3250
 	1    0    0    -1
@@
 F 0 "C11" H 7350 3350 50  0000 L CNN
 F 1 "100n" H 7350 3150 50  0000 L CNN
-F 2 "Capacitors_SMD:C_0603" H 7338 3100 30  0001 C CNN
-F 3 "http://psearch.en.murata.com/capacitor/product/GRM188R71E104KA01%23.pdf" H 7350 3350 60  0001 C CNN
+F 2 "Capacitors_SMD:C_0805" H 7338 3100 30  0001 C CNN
+F 3 "" H 7350 3350 60  0001 C CNN
 F 4 "Mouser" H 3650 5050 60  0001 C CNN "Supplier"
 F 5 "81-GRM39X104K25 " H 3650 5050 60  0001 C CNN "Supplier Part Number"

Commit message: Fix footprints
Parts:
- C13, C14: footprint Capacitors_SMD:C_0805 -> Capacitor_SMD:C_0805_2012Metric_Pad1.15x1.40mm_HandSolder
- D2: footprint Diodes_SMD:SOD-123 -> Diode_SMD:D_SOD-123
- Q1: footprint Housings_SOT-23_SOT-143_TSOT-6:SOT-23 -> Package_TO_SOT_SMD:SOT-23_Handsoldering
- R2, R3, R4, R5, R6: footprint Resistors_SMD:R_0805 -> Resistor_SMD:R_0805_2012Metric_Pad1.15x1.40mm_HandSolder
- REL1: footprint uMIDI-switcher:Omron_G6K-2P -> umidi-wah:Omron_G6K-2P
Changed lines of the file:
@@
 F 0 "REL1" H 8050 3500 60  0000 C CNN
 F 1 "Omron G6K-2P-5VCD" H 8050 3600 60  0000 C CNN
-F 2 "uMIDI-switcher:Omron_G6K-2P" H 8050 3300 60  0001 C CNN
+F 2 "umidi-wah:Omron_G6K-2P" H 8050 3300 60  0001 C CNN
 F 3 "https://www.omron.com/ecb/products/pdf/en-g6k.pdf" H 8050 3500 60  0001 C CNN
 F 4 "Mouser" H 8050 3500 60  0001 C CNN "Supplier"
@@
 F 0 "REL1" H 3700 4000 60  0000 C CNN
 F 1 "Omron G6K-2P-5VCD" H 3700 3500 60  0001 C CNN
-F 2 "uMIDI-switcher:Omron_G6K-2P" H 3700 3800 60  0001 C CNN
+F 2 "umidi-wah:Omron_G6K-2P" H 3700 3800 60  0001 C CNN
 F 3 "https://www.omron.com/ecb/products/pdf/en-g6k.pdf" H 3700 4000 60  0001 C CNN
 F 4 "Mouser" H 3700 4000 60  0001 C CNN "Supplier"
@@
 F 0 "REL1" H 5200 4000 60  0000 C CNN
 F 1 "Omron G6K-2P-5VCD" H 4850 4150 60  0001 C CNN
-F 2 "uMIDI-switcher:Omron_G6K-2P" H 5200 3800 60  0001 C CNN
+F 2 "umidi-wah:Omron_G6K-2P" H 5200 3800 60  0001 C CNN
 F 3 "https://www.omron.com/ecb/products/pdf/en-g6k.pdf" H 5200 4000 60  0001 C CNN
 F 4 "Mouser" H 5200 4000 60  0001 C CNN "Supplier"
@@
 F 0 "R16" V 4100 4150 50  0000 C CNN
 F 1 "100M" V 4200 4150 50  0000 C CNN
-F 2 "Resistors_SMD:R_0805" V 4130 4150 30  0001 C CNN
+F 2 "Resistor_SMD:R_0805_2012Metric_Pad1.15x1.40mm_HandSolder" V 4130 4150 30  0001 C CNN
 F 3 "" H 4100 4150 60  0001 C CNN
 	1    4200 4150
@@
 F 0 "D3" H 7750 3400 50  0000 C CNN
 F 1 "1N4148" H 7750 3200 50  0000 C CNN
-F 2 "Diodes_SMD:SOD-123" H 7750 3300 60  0001 C CNN
+F 2 "Diode_SMD:D_SOD-123" H 7750 3300 60  0001 C CNN
 F 3 "http://www.diodes.com/_files/datasheets/ds30086.pdf" H 7750 3400 60  0001 C CNN
 F 4 "Mouser" H 7750 3400 60  0001 C CNN "Supplier"
@@
 F 0 "C10" H 6650 3350 50  0000 L CNN
 F 1 "100n" H 6650 3150 50  0000 L CNN
-F 2 "Capacitors_SMD:C_0805" H 6638 3100 30  0001 C CNN
+F 2 "Capacitor_SMD:C_0805_2012Metric_Pad1.15x1.40mm_HandSolder" H 6638 3100 30  0001 C CNN
 F 3 "" H 6650 3350 60  0001 C CNN
 	1    6600 3250
@@
 F 0 "R20" V 7580 4600 50  0000 C CNN
 F 1 "10k" V 7507 4601 50  0000 C CNN
-F 2 "Resistors_SMD:R_0805" V 7430 4600 30  0001 C CNN
+F 2 "Resistor_SMD:R_0805_2012Metric_Pad1.15x1.40mm_HandSolder" V 7430 4600 30  0001 C CNN
 F 3 "" H 7580 4600 60  0001 C CNN
 F 4 "Mouser" H 7580 4600 60  0001 C CNN "Supplier"
@@
 F 0 "Q3" H 7800 4101 40  0000 R CNN
 F 1 "BSS138" H 7800 4400 40  0000 R CNN
-F 2 "Housings_SOT-23_SOT-143_TSOT-6:SOT-23" H 7670 4352 29  0001 C CNN
+F 2 "Package_TO_SOT_SMD:SOT-23_Handsoldering" H 7670 4352 29  0001 C CNN
 F 3 "https://www.fairchildsemi.com/datasheets/BS/BSS138.pdf" H 7800 4101 60  0001 C CNN
 F 4 "Mouser" H 3650 5050 60  0001 C CNN "Supplier"
@@
 F 0 "R19" V 6850 3000 50  0000 C CNN
 F 1 "180" V 6957 3001 50  0000 C CNN
-F 2 "Resistors_SMD:R_0805" V 6880 3000 30  0001 C CNN
+F 2 "Resistor_SMD:R_0805_2012Metric_Pad1.15x1.40mm_HandSolder" V 6880 3000 30  0001 C CNN
 F 3 "" H 6850 3000 60  0001 C CNN
 F 4 "Mouser" H 6850 3000 60  0001 C CNN "Supplier"
@@
 F 0 "C11" H 7350 3350 50  0000 L CNN
 F 1 "100n" H 7350 3150 50  0000 L CNN
-F 2 "Capacitors_SMD:C_0805" H 7338 3100 30  0001 C CNN
+F 2 "Capacitor_SMD:C_0805_2012Metric_Pad1.15x1.40mm_HandSolder" H 7338 3100 30  0001 C CNN
 F 3 "" H 7350 3350 60  0001 C CNN
 F 4 "Mouser" H 3650 5050 60  0001 C CNN "Supplier"
@@
 F 0 "R17" V 4350 4150 50  0000 C CNN
 F 1 "100M" V 4450 4150 50  0000 C CNN
-F 2 "Resistors_SMD:R_0805" V 4380 4150 30  0001 C CNN
+F 2 "Resistor_SMD:R_0805_2012Metric_Pad1.15x1.40mm_HandSolder" V 4380 4150 30  0001 C CNN
 F 3 "" H 4350 4150 60  0001 C CNN
 F 4 "Mouser" H 4350 4150 60  0001 C CNN "Supplier"
@@
 F 0 "R18" V 4600 4150 50  0000 C CNN
 F 1 "100M" V 4700 4150 50  0000 C CNN
-F 2 "Resistors_SMD:R_0805" V 4630 4150 30  0001 C CNN
+F 2 "Resistor_SMD:R_0805_2012Metric_Pad1.15x1.40mm_HandSolder" V 4630 4150 30  0001 C CNN
 F 3 "" H 4600 4150 60  0001 C CNN
 F 4 "Mouser" H 4600 4150 60  0001 C CNN "Supplier"
