File: hardware/bypass.sch (KiCad schematic (older format))
At the start: 11 parts, among them Q3 BC547

Commit message: Revision BOM: Get low-tech parts from Reichelt
Parts:
- C13, C14: Manufacturer (none) -> YAGEO; Manufacturer Part Number (none) -> CC0805KRX7R9BB104; Supplier RS -> Reichelt; Supplier Link https://de.rs-online.com/web/p/keramik-vielschichtkondensat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 -> https://www.reichelt.de/smd-vielschicht-keramikkondensator-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; Supplier Part Number 170-0041 -> X7R-G0805 100N
- D2: Manufacturer Diodes Zetex -> DIODES INCORPORATED; Manufacturer Link http://www.diodes.com/catalog/Switching_Diodes_5/1N4148W_28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 -> (none); Supplier RS -> Reichelt; Supplier Link https://de.rs-online.com/web/p/schaltdioden/7384728/ -> https://www.reichelt.de/schalt-diode-100-v-150-ma-sod-123-1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; Supplier Part Number 738-4728 -> 1N 4148W7F DII
- Q3: Manufacturer (none) -> DIOTEC; Manufacturer Part Number (none) -> BC547B; Supplier RS -> Reichelt; Supplier Link https://de.rs-online.com/web/p/bipolare-transistoren/166298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 -> https://www.reichelt.de/bipolartransistor-npn-45v-0-1a-0-5w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; Supplier Part Number 166-2988 -> BC 547B DIO
- R2, R3, R4, R6: Manufacturer (none) -> TE Connectivity; Manufacturer Part Number (none) -> RH73H2A100MKTN; Supplier Link https://de.rs-online.com/web/p/smd-widerstande/2945062/ -> https://www.rsonline-privat.de/Products/ProductDetail/TE-Co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; Supplier Part Number 294-5062 -> 2945062
- R5: Manufacturer Vishay/Dale -> YAGEO; Manufacturer Link http://www.vishay.com/resistors-fixed/list/product-20011/ -> (none); Manufacturer Part Number CRCW0805180RFKEA -> RC0805FR-07180RL; Supplier RS -> Reichelt; Supplier Link https://de.rs-online.com/web/p/smd-widerstande/6790942/ -> https://www.reichelt.de/smd-widerstand-0805-180-ohm-125-mw-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; Supplier Part Number 679-0942 -> SMD-0805 180
- R5: Manufacturer (none) -> YAGEO; Manufacturer Part Number (none) -> RC0805FR-071KL; Supplier RS -> Reichelt; Supplier Link https://de.rs-online.com/web/p/smd-widerstande/8046449/ -> https://www.reichelt.de/smd-widerstand-0805-1-0-kohm-125-mw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; Supplier Part Number 804-6449 -> SMD-0805 1,00K
- REL1: Supplier Link https://de.rs-online.com/web/p/monostabile-relais/3650440/ -> https://www.rsonline-privat.de/Products/ProductDetail/Omron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; Supplier Part Number 365-0440 -> 3650440

Commit message: Fix relais supply
Changed lines of the file:
@@
 $EndComp
-$Comp
-L power:+9V #PWR042
-U 1 1 54E940D4
-P 6350 2950
-AR Path="/56223A3E/54E940D4" Ref="#PWR042"  Part="1"
-AR Path="/56223A52/54E9BE9F/54E940D4" Ref="#PWR049"  Part="1"
-AR Path="/56223A60/54E9BE9F/54E940D4" Ref="#PWR056"  Part="1"
-AR Path="/56223A6E/54E9BE9F/54E940D4" Ref="#PWR063"  Part="1"
-AR Path="/56223A7C/54E9BE9F/54E940D4" Ref="#PWR070"  Part="1"
-AR Path="/56223A90/54E9BE9F/54E940D4" Ref="#PWR077"  Part="1"
-AR Path="/5CD91DFE/54E940D4" Ref="#PWR020"  Part="1"
-F 0 "#PWR020" H 6350 2800 60  0001 C CNN
-F 1 "+9V" H 6350 3090 60  0000 C CNN
-F 2 "" H 6350 2950 60  0000 C CNN
-F 3 "" H 6350 2950 60  0000 C CNN
-	1    6350 2950
-	1    0    0    -1
-$EndComp
-Wire Wire Line
-	6350 2950 6350 3000
 $Comp
 L uMIDI-wah-rescue:R-uMIDI-switcher-rescue R3
@@
 Text Label 4300 3900 0    60   ~ 0
 bypass
-Text Label 3150 3800 0    60   ~ 0
-loop_in
-Text Label 5450 3800 0    60   ~ 0
-loop_out
-Text Label 4200 3600 1    60   ~ 0
-fx_send
-Text Label 4700 3600 1    60   ~ 0
-fx_return
 Text Label 7350 3000 0    60   ~ 0
 relais_p
@@
 Wire Wire Line
 	6650 4250 7100 4250
+Text HLabel 6350 3000 0    50   Input ~ 0
++9V
 $EndSCHEMATC
