File: hardware/filter.kicad_sch (KiCad schematic)
At the start: 57 parts, among them J2 Pots Main, J3 Pots Front, Q1 KSC1815, Q2 KSC1815, U1 NJM4558D, U2 NJM4558D, U4 NJM4558D, U5 NJM4558D

Commit message: Replace bourns potentiometers in schematic and board
Parts:
- RV5: footprint uMidi-wah:Bourns PC Axial Rear Mounting Bracket -> uMidi-wah:Potentiometer_Alpha_RV16AF-20-15k-Single_Horizontal
Changed lines of the file:
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@@
       (effects (font (size 1.27 1.27)))
     )
-    (property "Footprint" "uMidi-wah:Bourns PC Axial Rear Mounting Bracket" (at 120.65 66.04 0)
+    (property "Footprint" "uMidi-wah:Potentiometer_Alpha_RV16AF-20-15k-Single_Horizontal" (at 120.65 66.04 0)
       (effects (font (size 1.27 1.27)) hide)
     )
@@
       (effects (font (size 1.27 1.27)))
     )
-    (property "Footprint" "uMidi-wah:Bourns PC Axial Rear Mounting Bracket" (at 154.94 48.26 0)
+    (property "Footprint" "uMidi-wah:Potentiometer_Alpha_RV16AF-20-15k-Single_Horizontal" (at 154.94 48.26 0)
       (effects (font (size 1.27 1.27)) hide)
     )
@@
       (effects (font (size 1.27 1.27)))
     )
-    (property "Footprint" "uMidi-wah:Bourns PC Axial Rear Mounting Bracket" (at 171.45 92.71 0)
+    (property "Footprint" "uMidi-wah:Potentiometer_Alpha_RV16AF-20-15k-Single_Horizontal" (at 171.45 92.71 0)
       (effects (font (size 1.27 1.27)) hide)
     )
@@
       (effects (font (size 1.27 1.27)))
     )
-    (property "Footprint" "uMidi-wah:Bourns PC Axial Rear Mounting Bracket" (at 121.92 110.49 0)
-      (effects (font (size 1.27 1.27)) hide)
-    )
+    (property "Footprint" "uMidi-wah:Potentiometer_Alpha_RV16AF-20-15k-Single_Horizontal" (at 121.92 110.49 0)
+      (effects (font (size 1.27 1.27)) hide)
+    )

Commit message: Add some supplier links and datasheets
Parts:
- Q1, Q2: Manufacturer (none) -> On Semi; Manufacturer Part Number (none) -> KSC1815; Supplier (none) -> Mouser; Supplier Link (none) -> https://www.mouser.de/ProductDetail/onsemi-Fairchild/KSC181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
- R20, R26: Supplier (none) -> Mouser; Supplier Link (none) -> https://www.mouser.de/ProductDetail/Amphenol-Piher/PT10LV10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
- R22: Supplier Digikey -> Mouser; Supplier Link (none) -> https://www.mouser.de/ProductDetail/Advanced-Photonix/PDV-P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
- RV5: Supplier (none) -> Mouser
- RV5: Supplier (none) -> Conrad, Voelkner
- U1, U2, U4, U5: Manufacturer (none) -> Nisshinbo / JRC; Manufacturer Part Number (none) -> NJM4558D; Supplier (none) -> Mouser; Supplier Link (none) -> https://www.mouser.de/ProductDetail/Nisshinbo/NJM4558D?qs=u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

Commit message: Add supplier link; Change footprint of 18n film cap
Parts:
- C12: footprint Capacitor_THT:C_Rect_L4.6mm_W5.5mm_P2.50mm_MKS02_FKP02 -> Capacitor_THT:C_Rect_L7.0mm_W2.5mm_P5.00mm; Manufacturer (none) -> Kemet; Supplier (none) -> Mouser; Supplier Link (none) -> https://www.mouser.de/ProductDetail/KEMET/MMK5183J50J01L4BU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
- C2, C22: Manufacturer (none) -> WIMA; Supplier (none) -> Mouser; Supplier Link (none) -> https://www.mouser.de/ProductDetail/WIMA/MKS2B051001N00JSSD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
- C8: Supplier (none) -> Mouser; Supplier Link (none) -> https://www.mouser.de/ProductDetail/WIMA/MKS02-1-50-10?qs=o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
Changed lines of the file:
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@@
       (effects (font (size 1.27 1.27)) hide)
     )
-    (property "Supplier Link" "" (at 72.39 95.25 0)
+    (property "Supplier Link" "https://www.mouser.de/ProductDetail/WIMA/MKS02-1-50-10?qs=olJun0bQHM94q8okHP6KHQ%3D%3D" (at 72.39 95.25 0)
+      (effects (font (size 1.27 1.27)) hide)
+    )
+    (property "Supplier" "Mouser" (at 72.39 95.25 0)
       (effects (font (size 1.27 1.27)) hide)
     )
@@
       (effects (font (size 1.27 1.27)) hide)
     )
-    (property "Datasheet" "~" (at 27.305 88.9 0)
-      (effects (font (size 1.27 1.27)) hide)
-    )
-    (property "Supplier Link" "" (at 27.305 88.9 0)
+    (property "Datasheet" "https://www.mouser.de/datasheet/2/440/e_WIMA_MKS_2-1139871.pdf" (at 27.305 88.9 0)
+      (effects (font (size 1.27 1.27)) hide)
+    )
+    (property "Supplier Link" "https://www.mouser.de/ProductDetail/WIMA/MKS2B051001N00JSSD?qs=sJjjjplDs9sVDxmbrDbs4Q%3D%3D" (at 27.305 88.9 0)
+      (effects (font (size 1.27 1.27)) hide)
+    )
+    (property "Manufacturer" "WIMA" (at 27.305 88.9 0)
+      (effects (font (size 1.27 1.27)) hide)
+    )
+    (property "Supplier" "Mouser" (at 27.305 88.9 0)
       (effects (font (size 1.27 1.27)) hide)
     )
@@
       (effects (font (size 1.27 1.27)))
     )
-    (property "Footprint" "Capacitor_THT:C_Rect_L4.6mm_W5.5mm_P2.50mm_MKS02_FKP02" (at 107.95 105.7148 0)
-      (effects (font (size 1.27 1.27)) hide)
-    )
-    (property "Datasheet" "~" (at 104.14 106.68 0)
-      (effects (font (size 1.27 1.27)) hide)
-    )
-    (property "Supplier Link" "" (at 104.14 106.68 0)
+    (property "Footprint" "Capacitor_THT:C_Rect_L7.0mm_W2.5mm_P5.00mm" (at 107.95 105.7148 0)
+      (effects (font (size 1.27 1.27)) hide)
+    )
+    (property "Datasheet" "https://www.mouser.de/ProductDetail/WIMA/MKS02-1-50-10?qs=olJun0bQHM94q8okHP6KHQ%3D%3D" (at 104.14 106.68 0)
+      (effects (font (size 1.27 1.27)) hide)
+    )
+    (property "Supplier Link" "https://www.mouser.de/ProductDetail/KEMET/MMK5183J50J01L4BULK?qs=IKDMbYZLynA%252BvMsRrHXlyg%3D%3D" (at 104.14 106.68 0)
+      (effects (font (size 1.27 1.27)) hide)
+    )
+    (property "Manufacturer" "Kemet" (at 104.14 106.68 0)
+      (effects (font (size 1.27 1.27)) hide)
+    )
+    (property "Supplier" "Mouser" (at 104.14 106.68 0)
       (effects (font (size 1.27 1.27)) hide)
     )
@@
       (effects (font (size 1.27 1.27)) hide)
     )
-    (property "Datasheet" "~" (at 262.89 69.85 0)
-      (effects (font (size 1.27 1.27)) hide)
-    )
-    (property "Supplier Link" "" (at 262.89 69.85 0)
-      (effects (font (size 1.27 1.27)) hide)
-    )
+    (property "Datasheet" "https://www.mouser.de/datasheet/2/440/e_WIMA_MKS_2-1139871.pdf" (at 262.89 69.85 0)
+      (effects (font (size 1.27 1.27)) hide)
+    )
+    (property "Supplier Link" "https://www.mouser.de/ProductDetail/WIMA/MKS2B051001N00JSSD?qs=sJjjjplDs9sVDxmbrDbs4Q%3D%3D" (at 262.89 69.85 0)
+      (effects (font (size 1.27 1.27)) hide)
+    )
+    (property "Manufacturer" "WIMA" (at 262.89 69.85 0)
+      (effects (font (size 1.27 1.27)) hide)
+    )
+    (property "Supplier" "Mouser" (at 262.89 69.85 0)
+      (effects (font (size 1.27 1.27)) hide)
+    )

Commit message: Specify 2n7 foil cap; Use generic 2.5/5mm footprints
Parts:
- C12: footprint Capacitor_THT:C_Rect_L7.0mm_W2.5mm_P5.00mm -> Capacitor_THT:C_Rect_L7.0mm_W3.5mm_P2.50mm_P5.00mm
- C14: Manufacturer (none) -> WIMA; Manufacturer Part Number (none) -> MKS0C021000B00JSSD; Supplier (none) -> Mouser; Supplier Link (none) -> https://www.mouser.de/ProductDetail/WIMA/MKS0C021000B00JSSD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
- C17: footprint Capacitor_THT:C_Rect_L4.6mm_W5.5mm_P2.50mm_MKS02_FKP02 -> Capacitor_THT:C_Rect_L7.0mm_W3.5mm_P2.50mm_P5.00mm; Manufacturer (none) -> Kemet; Supplier (none) -> Mouser; Supplier Link (none) -> https://www.mouser.de/ProductDetail/KEMET/MMK5272K63J01L16.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
Changed lines of the file:
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@@
       (effects (font (size 1.27 1.27)))
     )
-    (property "Footprint" "Capacitor_THT:C_Rect_L7.0mm_W2.5mm_P5.00mm" (at 107.95 105.7148 0)
+    (property "Footprint" "Capacitor_THT:C_Rect_L7.0mm_W3.5mm_P2.50mm_P5.00mm" (at 107.95 105.7148 0)
       (effects (font (size 1.27 1.27)) hide)
     )
@@
       (effects (font (size 1.27 1.27)))
     )
-    (property "Footprint" "Capacitor_THT:C_Rect_L4.6mm_W5.5mm_P2.50mm_MKS02_FKP02" (at 203.2 79.0448 0)
-      (effects (font (size 1.27 1.27)) hide)
-    )
-    (property "Datasheet" "~" (at 199.39 80.01 0)
-      (effects (font (size 1.27 1.27)) hide)
-    )
-    (property "Supplier Link" "" (at 199.39 80.01 0)
+    (property "Footprint" "Capacitor_THT:C_Rect_L7.0mm_W3.5mm_P2.50mm_P5.00mm" (at 203.2 79.0448 0)
+      (effects (font (size 1.27 1.27)) hide)
+    )
+    (property "Datasheet" "https://www.mouser.de/datasheet/2/212/F3294_MMK-1101858.pdf" (at 199.39 80.01 0)
+      (effects (font (size 1.27 1.27)) hide)
+    )
+    (property "Supplier Link" "https://www.mouser.de/ProductDetail/KEMET/MMK5272K63J01L16.5TA18?qs=IKDMbYZLynDZFzWwgE8yZQ%3D%3D" (at 199.39 80.01 0)
+      (effects (font (size 1.27 1.27)) hide)
+    )
+    (property "Supplier" "Mouser" (at 199.39 80.01 0)
+      (effects (font (size 1.27 1.27)) hide)
+    )
+    (property "Manufacturer" "Kemet" (at 199.39 80.01 0)
       (effects (font (size 1.27 1.27)) hide)
     )
@@
       (effects (font (size 1.27 1.27)) hide)
     )
-    (property "Datasheet" "~" (at 108.966 52.07 0)
-      (effects (font (size 1.27 1.27)) hide)
-    )
-    (property "Supplier Link" "" (at 108.966 52.07 0)
-      (effects (font (size 1.27 1.27)) hide)
-    )
+    (property "Datasheet" "https://www.mouser.de/datasheet/2/440/e_WIMA_MKS_02-1139783.pdf" (at 108.966 52.07 0)
+      (effects (font (size 1.27 1.27)) hide)
+    )
+    (property "Supplier Link" "https://www.mouser.de/ProductDetail/WIMA/MKS0C021000B00JSSD?qs=OiDNLlGUHG0VuoIdnA6lwg%3D%3D" (at 108.966 52.07 0)
+      (effects (font (size 1.27 1.27)) hide)
+    )
+    (property "Manufacturer" "WIMA" (at 108.966 52.07 0)
+      (effects (font (size 1.27 1.27)) hide)
+    )
+    (property "Manufacturer Part Number" "MKS0C021000B00JSSD " (at 108.966 52.07 0)
+      (effects (font (size 1.27 1.27)) hide)
+    )
+    (property "Supplier" "Mouser" (at 108.966 52.07 0)
+      (effects (font (size 1.27 1.27)) hide)
+    )

Commit message: Specify 47n cap
Parts:
- C20: Manufacturer (none) -> WIMA; Manufacturer Part Number (none) -> MKS0C024700B00JSSD; Supplier (none) -> Mouser; Supplier Link (none) -> https://www.mouser.de/ProductDetail/WIMA/MKS0C024700B00JSSD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
Changed lines of the file:
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@@
       (effects (font (size 1.27 1.27)) hide)
     )
-    (property "Datasheet" "~" (at 217.17 63.5 0)
+    (property "Datasheet" "https://www.mouser.de/datasheet/2/440/e_WIMA_MKS_02-1139783.pdf" (at 217.17 63.5 0)
       (effects (font (size 1.27 1.27)) hide)
     )
-    (property "Supplier Link" "" (at 217.17 63.5 0)
+    (property "Supplier Link" "https://www.mouser.de/ProductDetail/WIMA/MKS0C024700B00JSSD?qs=mjnqRw4WRuav7NfFCTGieQ%3D%3D" (at 217.17 63.5 0)
       (effects (font (size 1.27 1.27)) hide)
     )
+    (property "Manufacturer" "WIMA" (at 217.17 63.5 0)
+      (effects (font (size 1.27 1.27)) hide)
+    )
+    (property "Manufacturer Part Number" "MKS0C024700B00JSSD " (at 217.17 63.5 0)
+      (effects (font (size 1.27 1.27)) hide)
+    )
+    (property "Supplier" "Mouser" (at 217.17 63.5 0)
+      (effects (font (size 1.27 1.27)) hide)
+    )

Commit message: Review PCB
Connections:
- net status_led: no longer J2.10 (Pin_10), J3.10 (Pin_10)
- net at D3.2 (A), R24.1: now also J2.10 (Pin_10), J3.10 (Pin_10)
Other:
- moved on the sheet: D3, R24
Changed lines of the file:
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@@
   (junction (at 108.966 38.1) (diameter 0) (color 0 0 0 0)
   )
+  (junction (at 219.075 136.525) (diameter 0) (color 0 0 0 0)
+  )
   (junction (at 243.205 126.365) (diameter 0) (color 0 0 0 0)
   )
@@
   (junction (at 46.355 110.49) (diameter 0) (color 0 0 0 0)
   )
-  (junction (at 229.235 136.525) (diameter 0) (color 0 0 0 0)
-  )
   (junction (at 140.97 66.04) (diameter 0) (color 0 0 0 0)
   )
@@
     (stroke (width 0) (type default))
   )
-  (wire (pts (xy 227.965 136.525) (xy 229.235 136.525))
+  (wire (pts (xy 217.805 127) (xy 219.075 127))
     (stroke (width 0) (type default))
   )
@@
     (stroke (width 0) (type default))
   )
-  (wire (pts (xy 229.235 136.525) (xy 243.205 136.525))
+  (wire (pts (xy 219.075 136.525) (xy 243.205 136.525))
     (stroke (width 0) (type default))
   )
@@
     (stroke (width 0) (type default))
   )
-  (wire (pts (xy 229.235 137.795) (xy 229.235 136.525))
+  (wire (pts (xy 219.075 128.27) (xy 219.075 127))
     (stroke (width 0) (type default))
   )
@@
     (stroke (width 0) (type default))
   )
-  (wire (pts (xy 229.235 146.05) (xy 229.235 145.415))
+  (wire (pts (xy 219.075 136.525) (xy 219.075 135.89))
     (stroke (width 0) (type default))
   )
@@
     (stroke (width 0) (type default))
   )
-  (wire (pts (xy 229.235 154.305) (xy 229.235 153.67))
+  (wire (pts (xy 219.075 144.78) (xy 219.075 144.145))
     (stroke (width 0) (type default))
   )
@@
     (effects (font (size 1.27 1.27)) (justify left))
   )
-  (hierarchical_label "status_led" (shape input) (at 227.965 136.525 180) (fields_autoplaced)
+  (hierarchical_label "status_led" (shape input) (at 217.805 127 180) (fields_autoplaced)
     (effects (font (size 1.27 1.27)) (justify right))
   )
@@
     )
   )
-  (symbol (lib_id "power:GND") (at 229.235 154.305 0) (unit 1)
+  (symbol (lib_id "power:GND") (at 219.075 144.78 0) (unit 1)
     (in_bom yes) (on_board yes) (dnp no) (fields_autoplaced)
-    (property "Reference" "#PWR0119" (at 229.235 160.655 0)
+    (property "Reference" "#PWR0119" (at 219.075 151.13 0)
       (effects (font (size 1.27 1.27)) hide)
     )
-    (property "Value" "GND" (at 229.235 159.385 0)
+    (property "Value" "GND" (at 219.075 149.86 0)
       (effects (font (size 1.27 1.27)))
     )
-    (property "Footprint" "" (at 229.235 154.305 0)
+    (property "Footprint" "" (at 219.075 144.78 0)
       (effects (font (size 1.27 1.27)) hide)
     )
-    (property "Datasheet" "" (at 229.235 154.305 0)
+    (property "Datasheet" "" (at 219.075 144.78 0)
       (effects (font (size 1.27 1.27)) hide)
     )
@@
     )
   )
-  (symbol (lib_id "Device:R") (at 229.235 141.605 180) (unit 1)
+  (symbol (lib_id "Device:R") (at 219.075 132.08 180) (unit 1)
     (in_bom yes) (on_board yes) (dnp no) (fields_autoplaced)
-    (property "Reference" "R24" (at 231.775 140.3349 0)
+    (property "Reference" "R24" (at 221.615 130.8099 0)
       (effects (font (size 1.27 1.27)) (justify right))
     )
-    (property "Value" "180" (at 231.775 142.8749 0)
+    (property "Value" "180" (at 221.615 133.3499 0)
       (effects (font (size 1.27 1.27)) (justify right))
     )
-    (property "Footprint" "Resistor_SMD:R_0805_2012Metric_Pad1.20x1.40mm_HandSolder" (at 231.013 141.605 90)
+    (property "Footprint" "Resistor_SMD:R_0805_2012Metric_Pad1.20x1.40mm_HandSolder" (at 220.853 132.08 90)
       (effects (font (size 1.27 1.27)) hide)
     )
-    (property "Datasheet" "~" (at 229.235 141.605 0)
+    (property "Datasheet" "~" (at 219.075 132.08 0)
       (effects (font (size 1.27 1.27)) hide)
     )
-    (property "Supplier Link" "" (at 229.235 141.605 0)
+    (property "Supplier Link" "" (at 219.075 132.08 0)
       (effects (font (size 1.27 1.27)) hide)
     )
@@
     )
   )
-  (symbol (lib_id "Device:LED") (at 229.235 149.86 90) (unit 1)
+  (symbol (lib_id "Device:LED") (at 219.075 140.335 90) (unit 1)
     (in_bom yes) (on_board yes) (dnp no) (fields_autoplaced)
-    (property "Reference" "D3" (at 233.045 150.1774 90)
+    (property "Reference" "D3" (at 222.885 140.6524 90)
       (effects (font (size 1.27 1.27)) (justify right))
     )
-    (property "Value" "LED" (at 233.045 152.7174 90)
+    (property "Value" "LED" (at 222.885 143.1924 90)
       (effects (font (size 1.27 1.27)) (justify right))
     )
-    (property "Footprint" "LED_THT:LED_D5.0mm" (at 229.235 149.86 0)
+    (property "Footprint" "LED_THT:LED_D5.0mm" (at 219.075 140.335 0)
       (effects (font (size 1.27 1.27)) hide)
     )
-    (property "Datasheet" "~" (at 229.235 149.86 0)
+    (property "Datasheet" "~" (at 219.075 140.335 0)
       (effects (font (size 1.27 1.27)) hide)
     )
-    (property "Supplier Link" "" (at 229.235 149.86 0)
+    (property "Supplier Link" "" (at 219.075 140.335 0)
       (effects (font (size 1.27 1.27)) hide)
     )

Commit message: Increase trace widths (and more brd optimization)
Parts:
- renumbered R12 to R11, R11 to R12, R18 to R17, R17 to R18, R21 to R20, R20 to R21, RV5 to RV1, RV5 to RV2, RV5 to RV3, RV5 to RV4, U1 to U4, U2 to U5
